File: connectivity.kicad_sch (KiCad schematic)
At the start: 48 parts, among them CN1 GPS_Port, CN2 SM06B-GHS-TB(LF)(SN), J1 USB_C_Receptacle, U13 FT232RL, U16 DS1023-1X10SF11, U17 DS1023-1X8SF11, U18 DS1023-1X6SF11, U19 DS1023-1X8SF11, U21 DS1023-1X8SF11

Commit message: footprints, symbols kicad
Parts:
- removed CN1: GPS_Port, symbol SM06B-GHS-TB(LF)(SN)_1
- removed CN2: SM06B-GHS-TB(LF)(SN), symbol SM06B-GHS-TB(LF)(SN)
- removed F1: 04000025WR, symbol 04000025WR
- removed I2C1_CONN1: SM04B-GHS-TB(LF)(SN), symbol SM04B-GHS-TB(LF)(SN)
- removed I2C2_CONN1: SM04B-GHS-TB(LF)(SN), symbol SM04B-GHS-TB(LF)(SN)_1
- removed M_CONN1: ZX-PH2.0-6PWZ-Y, symbol ZX-PH2.0-6PWZ-Y
- removed M_CONN2: ZX-PH2.0-6PWZ-Y, symbol ZX-PH2.0-6PWZ-Y_1
- removed M_CONN3: ZX-PH2.0-6PWZ-Y, symbol ZX-PH2.0-6PWZ-Y_2
- removed M_CONN4: ZX-PH2.0-6PWZ-Y, symbol ZX-PH2.0-6PWZ-Y_3
- removed M_CONN5: ZX-PH2.0-6PWZ-Y, symbol ZX-PH2.0-6PWZ-Y_4
- removed M_CONN6: ZX-PH2.0-6PWZ-Y, symbol ZX-PH2.0-6PWZ-Y_5
- removed U13: FT232RL, symbol FT232RL
- removed U16: DS1023-1X10SF11, symbol DS1023-1X10SF11
- removed U17: DS1023-1X8SF11, symbol DS1023-1X8SF11
- removed U18: DS1023-1X6SF11, symbol DS1023-1X6SF11
- removed U19, U21: DS1023-1X8SF11, symbol DS1023-1X8SF11_1
- removed USB1: MICROUSB-5PIN, symbol MICROUSB-5PIN
- added CN2: GPS_Port, Connector_JST:JST_GH_SM06B-GHS-TB_1x06-1MP_P1.25mm_Horizontal, symbol MyLIB:SM_06B_GHS_TB
- added CN3: SM06B-GHS-TB(LF)(SN), Connector_JST:JST_GH_SM06B-GHS-TB_1x06-1MP_P1.25mm_Horizontal, symbol MyLIB:SM_06B_GHS_TB
- added Con1: DS1023-1X6SF11, Connector_PinHeader_1.00mm:PinHeader_1x06_P1.00mm_Vertical, symbol MyLIB:DS1023-1X6SF11
- added Con4: (no value), Connector_PinHeader_1.00mm:PinHeader_1x06_P1.00mm_Vertical, symbol MyLIB:Con
- added Con5, Con7: DS1023-1X8SF11, Connector_PinHeader_1.00mm:PinHeader_1x08_P1.00mm_Vertical, symbol MyLIB:DS1023-1X8SF11
- added Con6: DS1023-1X8SF11, Connector_PinHeader_1.00mm:PinHeader_1x06_P1.00mm_Vertical, symbol MyLIB:DS1023-1X8SF11
- added Con8: DS1023-1X10SF11, Connector_PinHeader_1.00mm:PinHeader_1x10_P1.00mm_Vertical, symbol MyLIB:DS1023-1X10SF11
- added Con9: (no value), Connector_PinHeader_1.00mm:PinHeader_1x12_P1.00mm_Vertical, symbol MyLIB:Con5
- added F3: 04000025WR, Fuse:Fuse_0603_1608Metric, symbol 04000025WR
- added I2C2_conn1, I2C2_conn2: SM04B-GHS-TB(LF)(SN), Connector_JST:JST_GH_SM04B-GHS-TB_1x04-1MP_P1.25mm_Horizontal, symbol MyLIB:I2C_connector
- added M_Con1, M_Con2, M_Con3, M_Con4, M_Con5, M_Con6: ZX-PH2.0-6PWZ-Y, symbol MyLIB:motor_con
- added U2: FT232RL, Package_SO:SSOP-28_5.3x10.2mm_P0.65mm, symbol MyLIB:FT232RL
- added USB2: MICROUSB-5PIN, Connector_USB:USB_Micro-B_GCT_USB3076-30-A, symbol MyLIB:microUSB
- C33, C34, C43, C7_TANTAL1: footprint (none) -> Capacitor_SMD:C_0603_1608Metric
- C41: value 4.7nF -> 0.01uF; footprint (none) -> Capacitor_SMD:C_0603_1608Metric
- Con2: footprint (none) -> Connector_PinHeader_1.00mm:PinHeader_1x04_P1.00mm_Vertical
- Con3: footprint (none) -> Connector_PinHeader_1.00mm:PinHeader_1x12_P1.00mm_Vertical
- DynamixelCon2: footprint (none) -> Connector_PinHeader_1.00mm:PinHeader_1x03_P1.00mm_Vertical
- F2: footprint (none) -> Fuse:Fuse_0603_1608Metric
- J1: footprint (none) -> Connector_USB:USB_C_Receptacle_JAE_DX07S024WJ1R350
- LED2, LED3, LED4, LED5: footprint (none) -> LED_SMD:LED_0603_1608Metric
- R23, R24, R25, R26, R27, R28, R29, R30, R42: footprint (none) -> Resistor_SMD:R_0805_2012Metric
- R43, R44: value 5.1k -> 6.8k; footprint (none) -> Resistor_SMD:R_0805_2012Metric
Connections:
- net +14.4v: now also M_Con1.3, M_Con2.3, M_Con3.3, M_Con4.3, M_Con5.3, M_Con6.3
- net +3v3: now also I2C2_conn1.1, I2C2_conn2.1, U2.17 (3V3OUT), U2.4 (VCCIO)
- net +5v: now also CN2.1, CN3.1, F3.1, U2.20 (VCC)
- net A0: now also Con6.1
- net A1: now also Con6.2
- net A2: now also Con6.3
- net A3: now also Con6.4
- net A4: now also Con6.5
- net A5: now also Con6.6
- net A6: now also Con6.7
- net A7: now also Con6.8
- net ADC(PA2): now also Con7.3
- net ADC(PA3): now also Con7.4
- net ADC(PA6): now also Con7.5
- net ADC(PA7): now also Con7.6
- net ADC(PC0): now also Con7.7
- net ADC(PC1): now also Con7.8
- net AVDD: now also Con8.3
- net CONN_M1_1: now also M_Con1.2
- net CONN_M1_2: now also M_Con1.1
- net CONN_M2_1: now also M_Con2.2
- net CONN_M2_2: now also M_Con2.1
- net CONN_M3_1: now also M_Con3.2
- net CONN_M3_2: now also M_Con3.1
- net CONN_M4_1: now also M_Con4.2
- net CONN_M4_2: now also M_Con4.1
- net CONN_M5_1: now also M_Con5.2
- net CONN_M5_2: now also M_Con5.1
- net CONN_M6_1: now also M_Con6.2
- net CONN_M6_2: now also M_Con6.1
- net DAC(PA4): now also Con7.1
- net DAC(PA5): now also Con7.2
- net ENC_A_M1: now also Con9.2, M_Con1.5
- net ENC_A_M2: now also Con9.4, M_Con2.5
- net ENC_A_M3: now also Con9.6, M_Con3.5
- net ENC_A_M4: now also Con9.8, M_Con4.5
- net ENC_A_M5: now also Con9.10, M_Con5.5
- net ENC_A_M6: now also Con9.12, M_Con6.5
- net ENC_B_M1: now also Con9.1, M_Con1.4
- net ENC_B_M2: now also Con9.3, M_Con2.4
- net ENC_B_M3: now also Con9.5, M_Con3.4
- net ENC_B_M4: now also Con9.7, M_Con4.4
- net ENC_B_M5: now also Con9.9, M_Con5.4
- net ENC_B_M6: now also Con9.11, M_Con6.4
- net GND: now also CN2.6, CN3.6, Con4.1, Con8.4, I2C2_conn1.4, I2C2_conn2.4, M_Con1.6, M_Con2.6, M_Con3.6, M_Con4.6, M_Con5.6, M_Con6.6, U2.18 (GND), U2.21 (GND), U2.25 (AGND), U2.26 (TEST), U2.7 (GND), USB2.5 (GND), USB2.6 (EP), USB2.7 (EP), USB2.8 (EP), USB2.9 (EP)
- net I2C2_SCL: now also I2C2_conn2.2
- net I2C2_SDA: now also I2C2_conn2.3
- net I2C_SCL: now also Con8.1
- net I2C_SDA: now also Con8.2
- net IOREF: now also Con5.2
- net NRST: now also Con4.5, Con5.3
- net PC3(A2): now also Con1.3
- net PD14: now also Con8.8
- net PD15: now also Con8.9
- net PF10(A5): now also Con1.6
- net PF12: now also Con8.10
- net PF3(A3): now also Con1.4
- net PF5(A4): now also Con1.5
- net USART4_RX: now also CN2.3
- net USART4_TX: now also CN2.2
- net USBDM: now also U2.16 (USBDM), USB2.2 (D-)
- net USBDP: now also U2.15 (USBDP), USB2.3 (D+)
- net ext_RXD: now also U2.5 (RXD)
- net ext_TXD: now also U2.1 (TXD)
- net at R32.1: now also I2C2_conn1.2
- net at R31.1: now also CN2.4
- net at LED3.1: now also U2.22 (CBUS1)
- net at LED2.1: now also U2.23 (CBUS0)
- net at R34.1: now also I2C2_conn1.3
- net at R33.1: now also CN2.5
- new net: F3.2, USB2.1 (VBUS)
- new net PA15: Con4.2
- new net SWO: Con4.6
- new net TCK: Con4.3
- new net TMS: Con4.4
- no-connect marks 2 -> 3
Other:
- note added: "2 GND, 5 V - с силовой на вычислитель Принципиальная схема программатора для STM32F103 Добавить конннектор под анализатор (5X2) Предусмотреть крепежные отверстия для соединения с корпусом"
- note removed: "2 GND, 5 V - с силовой на вычислитель Принципиальная схема программатора для STM32F103 2 разных проекта сделать в kicad и загрузить на гитхаб (силовая плата и вычислительная) Добавить конннектор под анализатор (5X2) Предусмотреть крепежные отверстия для соединения с корпусом"
- moved on the sheet: Con3

Commit message: Add files via upload
Parts:
- removed C33: 0.1uF, Capacitor_SMD:C_0603_1608Metric, symbol 0805_C9900012713
- removed C34: 0.1uF, Capacitor_SMD:C_0603_1608Metric, symbol 0805_C9900012713_1
- removed C7_TANTAL1: 10uF, Capacitor_SMD:C_0603_1608Metric, symbol TANTALUM SMT CAPACITOR 330UF C
- removed Con1: DS1023-1X6SF11, Connector_PinHeader_1.00mm:PinHeader_1x06_P1.00mm_Vertical, symbol MyLIB:DS1023-1X6SF11
- removed Con2: (no value), Connector_PinHeader_1.00mm:PinHeader_1x04_P1.00mm_Vertical, symbol MyLIB:Con4
- removed Con3, Con9: (no value), Connector_PinHeader_1.00mm:PinHeader_1x12_P1.00mm_Vertical, symbol MyLIB:Con5
- removed Con5, Con7: DS1023-1X8SF11, Connector_PinHeader_1.00mm:PinHeader_1x08_P1.00mm_Vertical, symbol MyLIB:DS1023-1X8SF11
- removed Con6: DS1023-1X8SF11, Connector_PinHeader_1.00mm:PinHeader_1x06_P1.00mm_Vertical, symbol MyLIB:DS1023-1X8SF11
- removed Con8: DS1023-1X10SF11, Connector_PinHeader_1.00mm:PinHeader_1x10_P1.00mm_Vertical, symbol MyLIB:DS1023-1X10SF11
- removed F3: 04000025WR, Fuse:Fuse_0603_1608Metric, symbol 04000025WR
- removed LED2: red, LED_SMD:LED_0603_1608Metric, symbol INH-S1608BAG20TP-Y3_C9900012538
- removed LED3: green, LED_SMD:LED_0603_1608Metric, symbol INH-S1608BAG20TP-Y3_C9900012538_1
- removed LED4: led, LED_SMD:LED_0603_1608Metric, symbol INH-S1608BAG20TP-Y3_C9900012538_1
- removed LED5: led, LED_SMD:LED_0603_1608Metric, symbol INH-S1608BAG20TP-Y3_C9900012538
- removed M_Con1, M_Con2, M_Con3, M_Con4, M_Con5, M_Con6: ZX-PH2.0-6PWZ-Y, symbol MyLIB:motor_con
- removed R23: 100, Resistor_SMD:R_0805_2012Metric, symbol R_0603_EU_1
- removed R24: 100, Resistor_SMD:R_0805_2012Metric, symbol R_0603_EU
- removed R25: 330, Resistor_SMD:R_0805_2012Metric, symbol R_0603_EU
- removed R26: 330, Resistor_SMD:R_0805_2012Metric, symbol R_0603_EU_1
- removed R27: 1K5, Resistor_SMD:R_0805_2012Metric, symbol R_0603_EU_2
- removed R28: 1K5, Resistor_SMD:R_0805_2012Metric, symbol R_0603_EU_3
- removed R29: 1K5, Resistor_SMD:R_0805_2012Metric, symbol R_0603_EU_4
- removed R30: 1K5, Resistor_SMD:R_0805_2012Metric, symbol R_0603_EU_5
- removed R31: 0, symbol R_0603_EU_6
- removed R32: 0, symbol R_0603_EU_7
- removed R33: 0, symbol R_0603_EU_8
- removed R34: 0, symbol R_0603_EU_9
- added C10: 10uF, Capacitor_SMD:C_0603_1608Metric, symbol Device:C_Polarized
- added C53, C54: 0.1uF, Capacitor_SMD:C_0603_1608Metric, symbol Device:C
- added Con1: DS1023-1X2SF11, Connector_PinHeader_1.00mm:PinHeader_1x02_P1.00mm_Vertical, symbol MyLIB:Con_power
- added Con9: DS1023-1X10SF11, Connector_PinHeader_1.00mm:PinHeader_1x10_P1.00mm_Vertical, symbol MyLIB:DS1023-1X10SF11
- added D2: green, LED_SMD:LED_0603_1608Metric, symbol Device:LED
- added D3: red, LED_SMD:LED_0603_1608Metric, symbol Device:LED
- added D4, D5: led, LED_SMD:LED_0603_1608Metric, symbol Device:LED
- added F1: 04000025WR, Fuse:Fuse_0603_1608Metric, symbol Device:Fuse
- added J10, J9: DS1023-1X6SF11, Connector_PinHeader_1.00mm:PinHeader_1x06_P1.00mm_Vertical, symbol Connector:Conn_01x06_Pin
- added J11, J12, J14: DS1023-1X8SF11, Connector_PinHeader_1.00mm:PinHeader_1x08_P1.00mm_Vertical, symbol Connector:Conn_01x08_Pin
- added J13: DS1023-1X7SF11, Connector_PinHeader_1.00mm:PinHeader_1x07_P1.00mm_Vertical, symbol Connector:Conn_01x07_Pin
- added J2, J3, J4, J5, J6, J7: DS1023-1X5SF11, Connector_PinHeader_2.54mm:PinHeader_1x05_P2.54mm_Vertical, symbol Connector:Conn_01x05_Pin
- added J8: DS1023-1X9S21, Connector_PinHeader_1.00mm:PinHeader_1x09_P1.00mm_Vertical, symbol Connector:Conn_01x09_Pin
- added R14, R15, R18, R19: 21, Resistor_SMD:R_0805_2012Metric, symbol Device:R
- added R16, R17, R20, R21: 1K5, Resistor_SMD:R_0805_2012Metric, symbol Device:R
- added R22, R25: 330, Resistor_SMD:R_0805_2012Metric, symbol Device:R
- added R26, R27: 100, Resistor_SMD:R_0805_2012Metric, symbol Device:R
- added con2: DS1023-1X3SF11, Connector_PinHeader_1.00mm:PinHeader_1x03_P1.00mm_Vertical, symbol MyLIB:con_3
- Con4: value (none) -> DS1023-1X6SF11
Connections:
- net I2C2_SCL is gone; now on net I2C_SCL: I2C2_conn2.2
- net I2C2_SDA is gone; now on net I2C_SDA: I2C2_conn2.3
- net +3v3: now also C53.1, R16.1, R17.1, R20.1, R21.1, R22.1, R25.1, con2.1
- net +5v: now also C10.1, C54.1, F1.1, con2.2
- net A0: now also Con9.1
- net A1: now also Con9.2
- net A2: now also Con9.3
- net A3: now also Con9.4
- net A4: now also Con9.5
- net A5: now also Con9.6
- net A6: now also Con9.7
- net A7: now also Con9.8
- net D10: now also J9.2 (Pin_2)
- net D11: now also J9.3 (Pin_3)
- net D12: now also J9.4 (Pin_4)
- net D13: now also J9.5 (Pin_5)
- net D2: now also J8.3 (Pin_3)
- net D3: now also J8.4 (Pin_4)
- net D4: now also J8.5 (Pin_5)
- net D5: now also J8.6 (Pin_6)
- net D6: now also J8.7 (Pin_7)
- net D7: now also J8.8 (Pin_8)
- net D8: now also J8.9 (Pin_9)
- net D9: now also J9.1 (Pin_1)
- net DAC(PA4): now also Con9.9
- net DAC(PA5): now also Con9.10
- net GND: now also C10.2, C53.2, C54.2, D4.1 (K), D5.1 (K), con2.3
- net I2C_SCL: now also Con1.1, R14.2, R15.2, R16.2, R20.2
- net I2C_SDA: now also Con1.2, R17.2, R18.2, R19.2, R21.2
- net at USB2.1 (VBUS): now also F1.2
- net at I2C2_conn1.2: now also R15.1
- net at I2C2_conn1.3: now also R18.1
- net at CN2.4: now also R14.1
- net at CN2.5: now also R19.1
- net at U2.22 (CBUS1): now also D2.1 (K)
- net at U2.23 (CBUS0): now also D3.1 (K)
- net PA15 renamed JTDI
- net TCK renamed CLK
- net TMS renamed SWDIO
- net USART4_RX renamed USART7_RX
- net USART4_TX renamed USART7_TX
- net ext_RXD renamed UART8_RX
- net ext_TXD renamed UART8_TX
- new net: D3.2 (A), R25.2
- new net: D4.2 (A), R26.2
- new net: D2.2 (A), R22.2
- new net: D5.2 (A), R27.2
- new net D0: J8.1 (Pin_1)
- new net D1: J8.2 (Pin_2)
- new net D14: J9.6 (Pin_6)
- new net D15: J10.1 (Pin_1)
- new net D16: J10.2 (Pin_2)
- new net D17: J10.3 (Pin_3)
- new net D18: J10.4 (Pin_4)
- new net D19: J10.5 (Pin_5)
- new net D20: J10.6 (Pin_6)
- new net D21: J11.1 (Pin_1)
- new net D22: J11.2 (Pin_2)
- new net D23: J11.3 (Pin_3)
- new net D24: J11.4 (Pin_4)
- new net D25: J11.5 (Pin_5)
- new net D26: J11.6 (Pin_6)
- new net D27: J11.7 (Pin_7)
- new net D28: J11.8 (Pin_8)
- new net D29: J12.1 (Pin_1)
- new net D30: J12.2 (Pin_2)
- new net D31: J12.3 (Pin_3)
- new net D32: J12.4 (Pin_4)
- new net D33: J12.5 (Pin_5)
- new net D34: J12.6 (Pin_6)
- new net D35: J12.7 (Pin_7)
- new net D36: J12.8 (Pin_8)
- new net D37: J13.1 (Pin_1)
- new net D38: J13.2 (Pin_2)
- new net D39: J13.3 (Pin_3)
- new net D40: J13.4 (Pin_4)
- new net D41: J13.5 (Pin_5)
- new net D42: J13.6 (Pin_6)
- new net D43: J13.7 (Pin_7)
- new net D44: J14.1 (Pin_1)
- new net D45: J14.2 (Pin_2)
- new net D46: J14.3 (Pin_3)
- new net D47: J14.4 (Pin_4)
- new net D48: J14.5 (Pin_5), R27.1
- new net D49: J14.6 (Pin_6), R26.1
- new net D50: J14.7 (Pin_7)
- new net D51: J14.8 (Pin_8)
- new net ENC_A_M1_mk: J2.4 (Pin_4)
- new net ENC_A_M2_mk: J3.4 (Pin_4)
- new net ENC_A_M3_mk: J4.4 (Pin_4)
- new net ENC_A_M4_mk: J5.4 (Pin_4)
- new net ENC_A_M5_mk: J6.4 (Pin_4)
- new net ENC_A_M6_mk: J7.4 (Pin_4)
- new net ENC_B_M1_mk: J2.5 (Pin_5)
- new net ENC_B_M2_mk: J3.5 (Pin_5)
- new net ENC_B_M3_mk: J4.5 (Pin_5)
- new net ENC_B_M4_mk: J5.5 (Pin_5)
- new net ENC_B_M5_mk: J6.5 (Pin_5)
- new net ENC_B_M6_mk: J7.5 (Pin_5)
- new net FS1: J2.3 (Pin_3)
- new net FS2: J3.3 (Pin_3)
- new net FS3: J4.3 (Pin_3)
- new net FS4: J5.3 (Pin_3)
- new net FS5: J6.3 (Pin_3)
- new net FS6: J7.3 (Pin_3)
- new net IN1_M1: J2.1 (Pin_1)
- new net IN1_M2: J3.1 (Pin_1)
- new net IN1_M3: J4.1 (Pin_1)
- new net IN1_M4: J5.1 (Pin_1)
- new net IN1_M5: J6.1 (Pin_1)
- new net IN1_M6: J7.1 (Pin_1)
- new net IN2_M1: J2.2 (Pin_2)
- new net IN2_M2: J3.2 (Pin_2)
- new net IN2_M3: J4.2 (Pin_2)
- new net IN2_M4: J5.2 (Pin_2)
- new net IN2_M5: J6.2 (Pin_2)
- new net IN2_M6: J7.2 (Pin_2)
- no-connect marks 3 -> 37
Other:
- note added: "Верхняя сторона"
- note added: "Добавить конннектор под анализатор (5X2) Предусмотреть крепежные отверстия для соединения с корпусом"
- note added: "Левая сторона"
- note added: "Нижняя сторона"
- note added: "Правая сторона"
- note removed: "2 GND, 5 V - с силовой на вычислитель Принципиальная схема программатора для STM32F103 Добавить конннектор под анализатор (5X2) Предусмотреть крепежные отверстия для соединения с корпусом"
- moved on the sheet: C43, C44, Con4, DynamixelCon2, USB2

Commit message: Add files via upload
Parts:
- renumbered C41 to C36, C53 to C37, C54 to C38, C10 to C39, C44 to C40, C43 to C41, CN2 to CN1, CN3 to CN2, Con1 to Con2, Con9 to Con3, D2 to D4, D4 to D5, D5 to D6, DynamixelCon2 to DynamixelCon1, F2 to F1, F1 to F2, J2 to J10, J3 to J11, J4 to J12, J6 to J13, J7 to J14, J8 to J2, J13 to J3, J14 to J4, J9 to J5, J10 to J6, J11 to J7, J12 to J8, J5 to J9, R42 to R39, R43 to R40, R44 to R41, R16 to R42, R17 to R43, R14 to R44, R15 to R45, R19 to R46, R18 to R47, R25 to R48, R22 to R49, R20 to R50, R21 to R51, R26 to R52, R27 to R53, U2 to U3, USB2 to USB1, con2 to con1

Commit message: Add files via upload
Parts:
- C40: footprint (none) -> Capacitor_SMD:C_0603_1608Metric
- Con2: footprint Connector_PinHeader_1.00mm:PinHeader_1x02_P1.00mm_Vertical -> Connector_PinHeader_2.54mm:PinHeader_1x02_P2.54mm_Vertical
- Con3: footprint Connector_PinHeader_1.00mm:PinHeader_1x10_P1.00mm_Vertical -> Connector_PinHeader_2.54mm:PinHeader_1x10_P2.54mm_Vertical
- Con4, J5, J6: footprint Connector_PinHeader_1.00mm:PinHeader_1x06_P1.00mm_Vertical -> Connector_PinHeader_2.54mm:PinHeader_1x06_P2.54mm_Vertical
- DynamixelCon1, con1: footprint Connector_PinHeader_1.00mm:PinHeader_1x03_P1.00mm_Vertical -> Connector_PinHeader_2.54mm:PinHeader_1x03_P2.54mm_Vertical
- J2: footprint Connector_PinHeader_1.00mm:PinHeader_1x09_P1.00mm_Vertical -> Connector_PinHeader_2.54mm:PinHeader_1x09_P2.54mm_Vertical
- J3: footprint Connector_PinHeader_1.00mm:PinHeader_1x07_P1.00mm_Vertical -> Connector_PinHeader_2.54mm:PinHeader_1x07_P2.54mm_Vertical
- J4, J7, J8: footprint Connector_PinHeader_1.00mm:PinHeader_1x08_P1.00mm_Vertical -> Connector_PinHeader_2.54mm:PinHeader_1x08_P2.54mm_Vertical
Changed lines of the file:
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@@
 	)
 	(junction
-		(at 275.59 100.33)
-		(diameter 0)
-		(color 0 0 0 0)
-	)
-	(junction
 		(at 130.81 204.47)
 		(diameter 0)
@@
 	)
 	(junction
-		(at 273.05 100.33)
-		(diameter 0)
-		(color 0 0 0 0)
-	)
-	(junction
 		(at 53.34 66.04)
 		(diameter 0)
@@
 	(wire
 		(pts
-			(xy 271.78 100.33) (xy 273.05 100.33)
-		)
-		(stroke
-			(width 0)
-			(type default)
-		)
-	)
-	(wire
-		(pts
 			(xy 209.55 58.42) (xy 200.66 58.42)
 		)
@@
 	(wire
 		(pts
-			(xy 275.59 92.71) (xy 275.59 100.33)
-		)
-		(stroke
-			(width 0)
-			(type default)
-		)
-	)
-	(wire
-		(pts
 			(xy 218.44 53.34) (xy 217.17 53.34)
 		)
@@
 	(wire
 		(pts
-			(xy 273.05 92.71) (xy 273.05 100.33)
-		)
-		(stroke
-			(width 0)
-			(type default)
-		)
-	)
-	(wire
-		(pts
 			(xy 209.55 52.07) (xy 209.55 58.42)
 		)
@@
 	(wire
 		(pts
-			(xy 275.59 100.33) (xy 276.86 100.33)
+			(xy 271.78 100.33) (xy 276.86 100.33)
 		)
 		(stroke
@@
 	(wire
 		(pts
-			(xy 273.05 100.33) (xy 275.59 100.33)
-		)
-		(stroke
-			(width 0)
-			(type default)
-		)
-	)
-	(wire
-		(pts
 			(xy 313.69 137.16) (xy 308.61 137.16)
 		)
@@
 		)
 	)
-	(global_label "VDDA"
-		(shape input)
-		(at 273.05 92.71 90)
-		(fields_autoplaced yes)
-		(effects
-			(font
-				(size 1.27 1.27)
-			)
-			(justify left)
-		)
-		(property "Intersheetrefs" "${INTERSHEET_REFS}"
-			(at 273.05 85.0076 90)
-			(hide yes)
-			(show_name no)
-			(do_not_autoplace no)
-			(effects
-				(font
-					(size 1.27 1.27)
-				)
-				(justify left)
-			)
-		)
-	)
 	(global_label "UART8_TX"
 		(shape input)
@@
 		)
 	)
-	(global_label "IOREF"
-		(shape input)
-		(at 275.59 92.71 90)
-		(effects
-			(font
-				(size 1.27 1.27)
-			)
-			(justify left)
-		)
-		(property "Intersheetrefs" "${INTERSHEET_REFS}"
-			(at 275.59 92.71 90)
-			(hide yes)
-			(show_name no)
-			(do_not_autoplace no)
-			(effects
-				(font
-					(size 1.27 1.27)
-				)
-			)
-		)
-	)
 	(global_label "SWDIO"
 		(shape input)
@@
 			)
 		)
-		(property "Footprint" "Connector_PinHeader_1.00mm:PinHeader_1x06_P1.00mm_Vertical"
+		(property "Footprint" "Connector_PinHeader_2.54mm:PinHeader_1x06_P2.54mm_Vertical"
 			(at 255.27 219.71 0)
 			(hide yes)
@@
 			)
 		)
-		(property "Footprint" ""
+		(property "Footprint" "Capacitor_SMD:C_0603_1608Metric"
 			(at 313.69 52.07 0)
 			(hide yes)
@@
 			)
 		)
-		(property "Footprint" "Connector_PinHeader_1.00mm:PinHeader_1x03_P1.00mm_Vertical"
+		(property "Footprint" "Connector_PinHeader_2.54mm:PinHeader_1x03_P2.54mm_Vertical"
 			(at 267.97 102.87 0)
 			(hide yes)
@@
 			)
 		)
-		(property "Footprint" "Connector_PinHeader_1.00mm:PinHeader_1x02_P1.00mm_Vertical"
+		(property "Footprint" "Connector_PinHeader_2.54mm:PinHeader_1x02_P2.54mm_Vertical"
 			(at 316.23 153.67 0)
 			(hide yes)
@@
 			)
 		)
-		(property "Footprint" "Connector_PinHeader_1.00mm:PinHeader_1x06_P1.00mm_Vertical"
+		(property "Footprint" "Connector_PinHeader_2.54mm:PinHeader_1x06_P2.54mm_Vertical"
 			(at 317.5 124.46 0)
 			(hide yes)
@@
 			)
 		)
-		(property "Footprint" "Connector_PinHeader_1.00mm:PinHeader_1x07_P1.00mm_Vertical"
+		(property "Footprint" "Connector_PinHeader_2.54mm:PinHeader_1x07_P2.54mm_Vertical"
 			(at 255.27 152.4 0)
 			(hide yes)
@@
 			)
 		)
-		(property "Footprint" "Connector_PinHeader_1.00mm:PinHeader_1x08_P1.00mm_Vertical"
+		(property "Footprint" "Connector_PinHeader_2.54mm:PinHeader_1x08_P2.54mm_Vertical"
 			(at 255.27 171.45 0)
 			(hide yes)
@@
 			)
 		)
-		(property "Footprint" "Connector_PinHeader_1.00mm:PinHeader_1x09_P1.00mm_Vertical"
+		(property "Footprint" "Connector_PinHeader_2.54mm:PinHeader_1x09_P2.54mm_Vertical"
 			(at 214.63 181.61 0)
 			(hide yes)
@@
 			)
 		)
-		(property "Footprint" "Connector_PinHeader_1.00mm:PinHeader_1x06_P1.00mm_Vertical"
+		(property "Footprint" "Connector_PinHeader_2.54mm:PinHeader_1x06_P2.54mm_Vertical"
 			(at 255.27 203.2 0)
 			(hide yes)
@@
 			)
 		)
-		(property "Footprint" "Connector_PinHeader_1.00mm:PinHeader_1x03_P1.00mm_Vertical"
+		(property "Footprint" "Connector_PinHeader_2.54mm:PinHeader_1x03_P2.54mm_Vertical"
 			(at 340.36 43.18 0)
 			(hide yes)
@@
 			)
 		)
-		(property "Footprint" "Connector_PinHeader_1.00mm:PinHeader_1x08_P1.00mm_Vertical"
+		(property "Footprint" "Connector_PinHeader_2.54mm:PinHeader_1x08_P2.54mm_Vertical"
 			(at 304.8 196.85 0)
 			(hide yes)
@@
 			)
 		)
-		(property "Footprint" "Connector_PinHeader_1.00mm:PinHeader_1x08_P1.00mm_Vertical"
+		(property "Footprint" "Connector_PinHeader_2.54mm:PinHeader_1x08_P2.54mm_Vertical"
 			(at 304.8 173.99 0)
 			(hide yes)
@@
 			)
 		)
-		(property "Footprint" "Connector_PinHeader_1.00mm:PinHeader_1x10_P1.00mm_Vertical"
+		(property "Footprint" "Connector_PinHeader_2.54mm:PinHeader_1x10_P2.54mm_Vertical"
 			(at 317.5 100.33 0)
 			(hide yes)

Commit message: На компе сделать
Parts:
- added C42: 100nF, Capacitor_SMD:C_0603_1608Metric, symbol Device:C
- added C43: 1uF, Capacitor_SMD:C_0603_1608Metric, symbol Device:C
- added D7: led, LED_SMD:LED_0603_1608Metric, symbol Device:LED
- added R54: 330, Resistor_SMD:R_0805_2012Metric, symbol Device:R
- J1: footprint Connector_USB:USB_C_Receptacle_JAE_DX07S024WJ1R350 -> Connector_USB:USB_C_Receptacle_HRO_TYPE-C-31-M-12
Connections:
- net +3v3: now also C42.1, C43.1, R54.1
- net GND: now also C42.2, C43.2, D7.1 (K)
- new net: D7.2 (A), R54.2
Other:
- note added: "UART под общение"
- note added: "Сделать так, чтобы можно было общаться с мк через USB"
- note added: "Убрать МикроЮСБ"
