File: connectivity.kicad_sch (KiCad schematic)
At the start: 55 parts, among them CN1 GPS_Port, Con2 DS1023-1X2SF11, J1 USB_C_Receptacle, J10 DS1023-1X8SF11, J11 DS1023-1X5SF11, J12 DS1023-1X5SF11, J13 DS1023-1X5SF11, J14 DS1023-1X5SF11, J15 DS1023-1X5SF11, J16 DS1023-1X5SF11, J17 DS1023-1X5SF11, J2 JST_GH_SM06B-GHS-TB, J3 JST_GH_SM06B-GHS-TB, J4 JST_GH_SM06B-GHS-TB, J5 JST_GH_SM06B-GHS-TB, J6 DS1023-1X11S21, J7 DS1023-1X11S21, J8 DS1023-1X6SF11, J9 DS1023-1X11S21, U3 SN65HVD232, con1 DS1023-1X3SF11

Commit message: Дорожки
Connections:
- net I2C2_SDA: now also I2C2_conn4.2, R48.2; no longer I2C2_conn4.3, R49.2
- net I2C2_SLC: now also I2C2_conn4.3, R49.2; no longer I2C2_conn4.2, R48.2
- net UART8_RX: now also I2C2_conn1.2; no longer I2C2_conn1.3
- net UART8_TX: now also I2C2_conn1.3; no longer I2C2_conn1.2
Changed lines of the file:
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@@
 	)
 	(junction
+		(at 190.5 45.72)
+		(diameter 0)
+		(color 0 0 0 0)
+	)
+	(junction
 		(at 53.34 60.96)
 		(diameter 0)
@@
 	)
 	(junction
-		(at 190.5 45.72)
+		(at 195.58 48.26)
 		(diameter 0)
 		(color 0 0 0 0)
@@
 	)
 	(junction
-		(at 195.58 48.26)
-		(diameter 0)
-		(color 0 0 0 0)
-	)
-	(junction
 		(at 114.3 67.31)
 		(diameter 0)
@@
 	(wire
 		(pts
+			(xy 58.42 162.56) (xy 62.23 162.56)
+		)
+		(stroke
+			(width 0)
+			(type default)
+		)
+	)
+	(wire
+		(pts
 			(xy 261.62 156.21) (xy 265.43 156.21)
 		)
@@
 	(wire
 		(pts
-			(xy 195.58 48.26) (xy 186.69 48.26)
-		)
-		(stroke
-			(width 0)
-			(type default)
-		)
-	)
-	(wire
-		(pts
 			(xy 269.24 93.98) (xy 273.05 93.98)
 		)
@@
 	(wire
 		(pts
+			(xy 58.42 160.02) (xy 62.23 160.02)
+		)
+		(stroke
+			(width 0)
+			(type default)
+		)
+	)
+	(wire
+		(pts
 			(xy 219.71 170.18) (xy 223.52 170.18)
 		)
@@
 	(wire
 		(pts
-			(xy 58.42 160.02) (xy 62.23 160.02)
-		)
-		(stroke
-			(width 0)
-			(type default)
-		)
-	)
-	(wire
-		(pts
 			(xy 134.62 52.07) (xy 134.62 55.88)
 		)
@@
 	(wire
 		(pts
+			(xy 186.69 48.26) (xy 195.58 48.26)
+		)
+		(stroke
+			(width 0)
+			(type default)
+		)
+	)
+	(wire
+		(pts
+			(xy 186.69 45.72) (xy 190.5 45.72)
+		)
+		(stroke
+			(width 0)
+			(type default)
+		)
+	)
+	(wire
+		(pts
 			(xy 219.71 193.04) (xy 223.52 193.04)
 		)
@@
 	(wire
 		(pts
-			(xy 190.5 45.72) (xy 186.69 45.72)
-		)
-		(stroke
-			(width 0)
-			(type default)
-		)
-	)
-	(wire
-		(pts
 			(xy 50.8 59.69) (xy 53.34 59.69)
 		)
@@
 	(wire
 		(pts
-			(xy 58.42 162.56) (xy 62.23 162.56)
-		)
-		(stroke
-			(width 0)
-			(type default)
-		)
-	)
-	(wire
-		(pts
 			(xy 275.59 26.67) (xy 283.21 26.67)
 		)
@@
 	(global_label "UART8_RX"
 		(shape input)
-		(at 58.42 162.56 180)
+		(at 58.42 160.02 180)
 		(effects
 			(font
@@
 		)
 		(property "Intersheetrefs" "${INTERSHEET_REFS}"
-			(at 58.42 162.56 0)
+			(at 58.42 160.02 0)
 			(hide yes)
 			(show_name no)
@@
 	(global_label "I2C2_SLC"
 		(shape input)
-		(at 186.69 45.72 180)
+		(at 186.69 48.26 180)
 		(fields_autoplaced yes)
 		(effects
@@
 		)
 		(property "Intersheetrefs" "${INTERSHEET_REFS}"
-			(at 174.9358 45.72 0)
+			(at 174.9358 48.26 0)
 			(hide yes)
 			(show_name no)
@@
 	(global_label "UART8_TX"
 		(shape input)
-		(at 58.42 160.02 180)
+		(at 58.42 162.56 180)
 		(effects
 			(font
@@
 		)
 		(property "Intersheetrefs" "${INTERSHEET_REFS}"
-			(at 58.42 160.02 0)
+			(at 58.42 162.56 0)
 			(hide yes)
 			(show_name no)
@@
 	(global_label "I2C2_SDA"
 		(shape input)
-		(at 186.69 48.26 180)
+		(at 186.69 45.72 180)
 		(fields_autoplaced yes)
 		(effects
@@
 		)
 		(property "Intersheetrefs" "${INTERSHEET_REFS}"
-			(at 174.8753 48.26 0)
+			(at 174.8753 45.72 0)
 			(hide yes)
 			(show_name no)

Commit message: Iter2
Parts:
- removed J6, J7, J9: DS1023-1X11S21, Connector_PinHeader_2.54mm:PinHeader_1x11_P2.54mm_Vertical, symbol Connector:Conn_01x11_Pin
- removed J8: DS1023-1X6SF11, Connector_PinHeader_2.54mm:PinHeader_1x06_P2.54mm_Vertical, symbol Connector:Conn_01x06_Pin
- added A1: Arduino_UNO_R2, Module:Arduino_UNO_R2, symbol MCU_Module:Arduino_UNO_R2
- added J18: DS1023-1X6SF11, Connector_PinHeader_2.54mm:PinHeader_1x06_P2.54mm_Vertical, symbol Connector:Conn_01x06_Pin
- added J19: Conn_01x08_Pin, symbol Connector:Conn_01x08_Pin
- added J20: Conn_01x10_Pin, symbol Connector:Conn_01x10_Pin
- added J21: Conn_01x07_Pin, symbol Connector:Conn_01x07_Pin
- added J22: DS1023-1X8S21, Connector_PinHeader_2.54mm:PinHeader_1x08_P2.54mm_Vertical, symbol Connector:Conn_01x08_Pin
- added J23, J9: DS1023-1X4S21, Connector_PinHeader_2.54mm:PinHeader_1x04_P2.54mm_Vertical, symbol Connector:Conn_01x04_Pin
- added J6: DS1023-1X9S21, Connector_PinHeader_2.54mm:PinHeader_1x09_P2.54mm_Vertical, symbol Connector:Conn_01x09_Pin
Connections:
- net D37 is gone; now on net D31: R50.1
- net D38 is gone; now on net D32: R51.1
- net +3v3: now also J21.4 (Pin_4)
- net +5v: now also J21.5 (Pin_5), J21.7 (Pin_7)
- net A0: now also J18.1 (Pin_1)
- net A1: now also J18.2 (Pin_2)
- net A2: now also J18.3 (Pin_3)
- net A3: now also J18.4 (Pin_4)
- net A4: now also J18.5 (Pin_5)
- net A5: now also J18.6 (Pin_6)
- net D0: now also J22.1 (Pin_1)
- net D1: now also J22.2 (Pin_2)
- net D10: now also J6.3 (Pin_3)
- net D11: now also J6.4 (Pin_4)
- net D12: now also J6.5 (Pin_5)
- net D13: now also J6.6 (Pin_6)
- net D14: now also J6.7 (Pin_7)
- net D15: now also J6.8 (Pin_8)
- net D16: now also J6.9 (Pin_9)
- net D17: now also J23.1 (Pin_1)
- net D18: now also J23.2 (Pin_2)
- net D19: now also J23.3 (Pin_3)
- net D2: now also J22.3 (Pin_3)
- net D20: now also J23.4 (Pin_4)
- net D21: now also J19.6 (Pin_6)
- net D22: now also J19.5 (Pin_5)
- net D23: now also J19.4 (Pin_4)
- net D24: now also J19.3 (Pin_3)
- net D25: now also J19.1 (Pin_1)
- net D26: now also J20.10 (Pin_10)
- net D27: now also J20.9 (Pin_9)
- net D28: now also J20.8 (Pin_8)
- net D29: now also J9.1 (Pin_1)
- net D3: now also J22.4 (Pin_4)
- net D30: now also J9.2 (Pin_2)
- net D31: now also J9.3 (Pin_3)
- net D32: now also J9.4 (Pin_4)
- net D4: now also J22.5 (Pin_5)
- net D5: now also J22.6 (Pin_6)
- net D6: now also J22.7 (Pin_7)
- net D7: now also J22.8 (Pin_8)
- net D8: now also J6.1 (Pin_1)
- net D9: now also J6.2 (Pin_2)
- net GND: now also J20.4 (Pin_4), J21.6 (Pin_6)
- net I2C2_SDA: now also J20.2 (Pin_2)
- net I2C2_SLC: now also J20.1 (Pin_1)
- new net PWM_ard: J19.2 (Pin_2)
- new net SPI2_MISO: J20.6 (Pin_6)
- new net SPI2_MOSI: J20.7 (Pin_7)
- new net SPI2_SCK: J20.5 (Pin_5)
- new net UART7_RX: J19.8 (Pin_8)
- new net UART7_TX: J19.7 (Pin_7)
- new net VREF+: J20.3 (Pin_3)
Other:
- note added: "Верхняя сторона D29 - D32"
- note added: "Левая сторона D0 - D7"
- note added: "Нижняя сторона D8 - D16"
- note added: "Правая сторона D17 - D20"
- note removed: "Верхняя сторона D33 - D38"
- note removed: "Левая сторона D0 - D10"
- note removed: "Нижняя сторона D11 - D21"
- note removed: "Правая сторона D22 - D32"

Commit message: Trass
Parts:
- removed J10: DS1023-1X8SF11, Connector_PinHeader_2.54mm:PinHeader_1x08_P2.54mm_Vertical, symbol Connector:Conn_01x08_Pin
- removed J12, J13, J14, J15, J16, J17: DS1023-1X5SF11, Connector_PinHeader_2.54mm:PinHeader_1x05_P2.54mm_Vertical, symbol Connector:Conn_01x05_Pin
- removed J18: DS1023-1X6SF11, Connector_PinHeader_2.54mm:PinHeader_1x06_P2.54mm_Vertical, symbol Connector:Conn_01x06_Pin
- removed J19: Conn_01x08_Pin, symbol Connector:Conn_01x08_Pin
- removed J20: Conn_01x10_Pin, symbol Connector:Conn_01x10_Pin
- removed J21: Conn_01x07_Pin, symbol Connector:Conn_01x07_Pin
- removed J6: DS1023-1X9S21, Connector_PinHeader_2.54mm:PinHeader_1x09_P2.54mm_Vertical, symbol Connector:Conn_01x09_Pin
- added J11, J12: DS1023-2X10S21, Connector_PinHeader_2.54mm:PinHeader_2x10_P2.54mm_Vertical, symbol Connector:Conn_01x20_Pin
- added J7: DS1023-1X11S21, Connector_PinHeader_2.54mm:PinHeader_1x11_P2.54mm_Vertical, symbol Connector:Conn_01x11_Pin
- added JP4, JP5: Jumper_3_Open, Connector_PinHeader_2.54mm:PinHeader_1x03_P2.54mm_Vertical, symbol Jumper:Jumper_3_Open
- A1: footprint Module:Arduino_UNO_R2 -> CastomLibrary:Arduino_UNO_R2
- renumbered C34 to C32, C35 to C33, C36 to C34, C37 to C35, C38 to C36, C39 to C37, J11 to J10, J22 to J6, J9 to J8, J23 to J9
Connections:
- net +3v3: now also A1.2 (IOREF), A1.4 (3V3)
- net +5v: now also A1.5 (+5V)
- net A0: now also A1.9 (A0)
- net A1: now also A1.10 (A1)
- net A2: now also A1.11 (A2)
- net A3: now also A1.12 (A3)
- net A4: now also JP4.3 (B)
- net A5: now also JP5.3 (B)
- net A6: now also J7.3 (Pin_3)
- net D10: now also J7.5 (Pin_5)
- net D11: now also J7.6 (Pin_6)
- net D12: now also J7.7 (Pin_7)
- net D13: now also J7.8 (Pin_8)
- net D14: now also J7.9 (Pin_9)
- net D15: now also J7.10 (Pin_10)
- net D16: now also J7.11 (Pin_11)
- net D21: now also A1.17 (D2)
- net D22: now also A1.18 (D3)
- net D23: now also A1.19 (D4)
- net D24: now also A1.20 (D5)
- net D25: now also A1.22 (D7)
- net D26: now also A1.23 (D8)
- net D27: now also A1.24 (D9)
- net D28: now also A1.25 (D10)
- net D8: now also J7.1 (Pin_1)
- net D9: now also J7.4 (Pin_4)
- net DAC: now also J7.2 (Pin_2)
- net ENC_A_M1_mk: now also J11.7 (Pin_7)
- net ENC_A_M2_mk: now also J11.8 (Pin_8)
- net ENC_A_M3_mk: now also J11.18 (Pin_18)
- net ENC_A_M4_mk: now also J12.7 (Pin_7)
- net ENC_A_M5_mk: now also J12.8 (Pin_8)
- net ENC_A_M6_mk: now also J12.18 (Pin_18)
- net ENC_B_M1_mk: now also J11.9 (Pin_9)
- net ENC_B_M2_mk: now also J11.10 (Pin_10)
- net ENC_B_M3_mk: now also J11.20 (Pin_20)
- net ENC_B_M4_mk: now also J12.9 (Pin_9)
- net ENC_B_M5_mk: now also J12.10 (Pin_10)
- net ENC_B_M6_mk: now also J12.20 (Pin_20)
- net FS1: now also J11.5 (Pin_5)
- net FS2: now also J11.6 (Pin_6)
- net FS3: now also J11.16 (Pin_16)
- net FS4: now also J12.5 (Pin_5)
- net FS5: now also J12.6 (Pin_6)
- net FS6: now also J12.16 (Pin_16)
- net GND: now also A1.29 (GND), A1.6 (GND), A1.7 (GND)
- net I2C2_SDA: now also JP4.1 (A)
- net I2C2_SLC: now also JP5.1 (A)
- net IN1_M1: now also J11.1 (Pin_1)
- net IN1_M2: now also J11.2 (Pin_2)
- net IN1_M3: now also J11.12 (Pin_12)
- net IN1_M4: now also J12.1 (Pin_1)
- net IN1_M5: now also J12.2 (Pin_2)
- net IN1_M6: now also J12.12 (Pin_12)
- net IN2_M1: now also J11.3 (Pin_3)
- net IN2_M2: now also J11.4 (Pin_4)
- net IN2_M3: now also J11.14 (Pin_14)
- net IN2_M4: now also J12.3 (Pin_3)
- net IN2_M5: now also J12.4 (Pin_4)
- net IN2_M6: now also J12.14 (Pin_14)
- net NRST: now also A1.3 (~{RESET})
- net PWM_ard: now also A1.21 (D6)
- net SPI2_MISO: now also A1.27 (D12)
- net SPI2_MOSI: now also A1.26 (D11)
- net SPI2_SCK: now also A1.28 (D13)
- net UART7_RX: now also A1.15 (D0/RX)
- net UART7_TX: now also A1.16 (D1/TX)
- net VREF+: now also A1.30 (AREF)
- net at A1.13 (SDA/A4): now also JP4.2 (C)
- net at A1.14 (SCL/A5): now also JP5.2 (C)
- no-connect marks 21 -> 32
