File: plat_logic.kicad_sch (KiCad schematic)
At the start: 85 parts, among them SW1 Button-SMD-4.5x4.5x5.5, SW2 Button-SMD-4.5x4.5x5.5, U1 STM32F429ZITx, U2 USBLC6-2SC6, Y1 NX3225GD 8.000MHZ EXS00A-CG06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, Y2 NX3215SA-32.768KHZ-EXS00A-MU0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

Commit message: edit pins shem plat_logic
Parts:
- removed C29: 100nF, Capacitor_SMD:C_0603_1608Metric, symbol Device:C
- removed C35: 22pF, Capacitor_SMD:C_0603_1608Metric, symbol Device:C
- removed R20: 1k, Resistor_SMD:R_0603_1608Metric, symbol Device:R
- removed R34: 47, Resistor_SMD:R_0805_2012Metric, symbol Device:R
- removed R38: 27K, Resistor_SMD:R_0805_2012Metric, symbol Device:R
- R6: value 0 -> 1М
- R7: value 100K -> 330
- Y1: value NX3225GD 8.000MHZ EXS00A-CG06684 -> CSTNE8M00GH5L000R0 8.000MHZ; footprint Crystal:Crystal_SMD_3225-4Pin_3.2x2.5mm -> Crystal:Crystal_SMD_3215-2Pin_3.2x1.5mm
Connections:
- net D40 is gone; now on net ENC_A_M2_mk: U1.117 (PD3)
- net D41 is gone; now on net ENC_B_M2_mk: U1.118 (PD4)
- net D42 is gone; now on net D36: U1.119 (PD5)
- net D44 is gone; now on net D37: U1.123 (PD7)
- net D46 is gone; now on net D38: U1.125 (PG10)
- net D47 is gone; now on net D39: U1.126 (PG11)
- net D48 is gone; now on net IN2_M3: U1.128 (PG13)
- net D50 is gone; now on net FS3: U1.132 (PG15)
- net D51 is gone; now on net ENC_A_M3_mk: U1.134 (PB4)
- net JTDI is gone; now on net D35: U1.110 (PA15)
- net SWO is gone; now on net IN1_M3: U1.133 (PB3)
- net USART7_RX is gone; now on net D19: U1.58 (PE7)
- net USART7_TX is gone; now on net D20: U1.59 (PE8)
- net +3v3: now also C11.2, C13.2, C14.2, C15.2, C16.2, C17.2, C18.2, C19.2, C21.2, C24.2, U1.108 (VDD), U1.121 (VDD), U1.131 (VDD), U1.144 (VDD), U1.17 (VDD), U1.30 (VDD), U1.39 (VDD), U1.52 (VDD), U1.62 (VDD), U1.72 (VDD), U1.84 (VDD), U1.95 (VDD); no longer C11.1, C13.1, C14.1, C15.1, C16.1, C17.1, C18.1, C19.1, C21.1, C24.1
- net A3: now also C27.2; no longer C27.1
- net D10: now also U1.27 (PC1); no longer U1.50 (PF12)
- net D11: now also U1.37 (PA3); no longer U1.53 (PF13)
- net D12: now also U1.49 (PF11); no longer U1.54 (PF14)
- net D13: now also U1.50 (PF12); no longer U1.55 (PF15)
- net D14: now also U1.53 (PF13); no longer U1.56 (PG0)
- net D15: now also U1.54 (PF14); no longer U1.57 (PG1)
- net D16: now also U1.55 (PF15); no longer U1.63 (PE10)
- net D17: now also U1.56 (PG0); no longer U1.65 (PE12)
- net D18: now also U1.57 (PG1); no longer U1.66 (PE13)
- net D19: no longer U1.67 (PE14)
- net D20: no longer U1.68 (PE15)
- net D21: now also U1.63 (PE10); no longer U1.78 (PD9)
- net D22: now also U1.73 (PB12); no longer U1.79 (PD10)
- net D23: now also U1.74 (PB13); no longer U1.80 (PD11)
- net D24: now also U1.79 (PD10); no longer U1.85 (PD14)
- net D25: now also U1.80 (PD11); no longer U1.86 (PD15)
- net D26: now also U1.81 (PD12); no longer U1.87 (PG2)
- net D27: now also U1.82 (PD13); no longer U1.88 (PG3)
- net D28: now also U1.85 (PD14); no longer U1.89 (PG4)
- net D29: now also U1.86 (PD15); no longer U1.90 (PG5)
- net D3: now also U1.4 (PE5); no longer U1.7 (PC13)
- net D30: now also U1.87 (PG2); no longer U1.91 (PG6)
- net D31: now also U1.88 (PG3); no longer U1.92 (PG7)
- net D32: now also U1.89 (PG4); no longer U1.93 (PG8)
- net D33: now also U1.90 (PG5); no longer U1.98 (PC8)
- net D34: now also U1.91 (PG6); no longer U1.99 (PC9)
- net D35: no longer U1.100 (PA8)
- net D36: no longer U1.102 (PA10)
- net D37: no longer U1.114 (PD0)
- net D38: no longer U1.115 (PD1)
- net D39: no longer U1.116 (PD2)
- net D4: now also U1.5 (PE6); no longer U1.12 (PF2)
- net D5: now also U1.7 (PC13); no longer U1.13 (PF3)
- net D6: now also U1.12 (PF2); no longer U1.14 (PF4)
- net D7: now also U1.21 (PF9); no longer U1.15 (PF5)
- net D9: now also U1.26 (PC0); no longer U1.49 (PF11)
- net Data: now also D1.5 (2A)
- net ENC_A_M1_mk: now also R14.1, U1.96 (PC6); no longer R13.2, U1.60 (PE9)
- net ENC_A_M2_mk: no longer U1.34 (PA0)
- net ENC_A_M3_mk: no longer U1.42 (PA6)
- net ENC_A_M4_mk: now also U1.136 (PB6); no longer U1.81 (PD12)
- net ENC_A_M5_mk: now also U1.34 (PA0); no longer U1.96 (PC6)
- net ENC_A_M6_mk: now also U1.60 (PE9); no longer U1.4 (PE5)
- net ENC_B_M1_mk: now also R13.2, U1.97 (PC7); no longer R14.1, U1.64 (PE11)
- net ENC_B_M2_mk: no longer U1.35 (PA1)
- net ENC_B_M3_mk: now also U1.135 (PB5); no longer U1.43 (PA7)
- net ENC_B_M4_mk: now also U1.137 (PB7); no longer U1.82 (PD13)
- net ENC_B_M5_mk: now also U1.35 (PA1); no longer U1.97 (PC7)
- net ENC_B_M6_mk: now also U1.64 (PE11); no longer U1.5 (PE6)
- net FS1: now also U1.93 (PG8); no longer U1.140 (PB9)
- net FS2: now also U1.78 (PD9); no longer U1.69 (PB10)
- net FS3: no longer U1.70 (PB11)
- net FS4: now also U1.18 (PF6); no longer U1.73 (PB12)
- net FS5: now also U1.28 (PC2); no longer U1.74 (PB13)
- net FS6: now also U1.68 (PE15); no longer U1.77 (PD8)
- net GND: now also C11.1, C12.2, C13.1, C14.1, C15.1, C16.1, C17.1, C18.1, C19.1, C21.1, C24.1, C27.1; no longer C27.2
- net IN1_M3: no longer U1.18 (PF6)
- net IN1_M5: now also U1.36 (PA2); no longer U1.20 (PF8)
- net IN1_M6: now also U1.70 (PB11); no longer U1.21 (PF9)
- net IN2_M1: now also U1.92 (PG7); no longer U1.46 (PB0)
- net IN2_M2: now also U1.77 (PD8); no longer U1.47 (PB1)
- net IN2_M3: no longer U1.135 (PB5)
- net IN2_M4: now also U1.20 (PF8); no longer U1.136 (PB6)
- net IN2_M5: now also U1.29 (PC3); no longer U1.137 (PB7)
- net IN2_M6: now also U1.69 (PB10); no longer U1.139 (PB8)
- net PH0: now also C2.2, Y1.2
- net PH1: now also R6.2
- net TX_Enable(Dynamixel_TTL): no longer U1.113 (PC12)
- net USART4_RX(Dynamixel_TTL): no longer U1.112 (PC11)
- net USART1_TX: now reaches U1.101 (PA9)
- net at U1.103 (PA11): now also U2.1 (I/O1); no longer U2.3 (I/O2)
- net at U1.104 (PA12): now also U2.3 (I/O2); no longer U2.1 (I/O1)
- net at R25.2: now also U1.13 (PF3); no longer U1.26 (PC0)
- net at R26.2: now also U1.14 (PF4); no longer U1.27 (PC1)
- net at R27.2: now also U1.15 (PF5); no longer U1.28 (PC2)
- net at R32.2: now also U1.44 (PC4); no longer U1.29 (PC3)
- net at R33.2: now also U1.47 (PB1); no longer U1.36 (PA2)
- net at R35.2: now also U1.45 (PC5); no longer U1.44 (PC4)
- net at R36.2: now also U1.46 (PB0); no longer U1.45 (PC5)
- net D43 renamed SPI3_MOSI
- net D45 renamed USART6_RX
- net D49 renamed USART6_TX
- net DAC(PA4) renamed DAC
- net DAC(PA5) renamed SPI1_SCK
- net I2C_SCL renamed I2C2_SLC
- net I2C_SDA renamed I2C2_SDA
- net USART4_TX(Dynamixel_TTL) renamed SPI3_SCK
- net SPI3_SCK: no longer D1.5 (2A)
- net USBDM(PA12) renamed USB_DP
- net USBDP(PA11) renamed USB_DM
- new net CAN1_RX: U1.114 (PD0)
- new net CAN1_TX: U1.115 (PD1)
- new net I2C1_SCL: U1.139 (PB8)
- new net I2C1_SDA: U1.140 (PB9)
- new net I2C3_SCL: U1.100 (PA8)
- new net I2C3_SDA: U1.99 (PC9)
- new net SDIO_CK: U1.113 (PC12)
- new net SDIO_CMD: U1.116 (PD2)
- new net SDIO_D0: U1.98 (PC8)
- new net SPI1_MISO: U1.42 (PA6)
- new net SPI1_MOSI: U1.43 (PA7)
- new net SPI3_MISO: U1.112 (PC11)
- new net SPI4_MISO: U1.66 (PE13)
- new net SPI4_MOSI: U1.67 (PE14)
- new net SPI4_SCK: U1.65 (PE12)
- new net USART1_RX: U1.102 (PA10)
Other:
- note removed: "Заменить из ТГ"
- note removed: "Когда в CubeMX делаешь PB4 GPIO_Input\Output, то JTAG(4 pins) сбрасывается почему-то"
- moved on the sheet: C10, C11, C12, C13, C14, C15, C16, C17, C18, C19, C20, C21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

Commit message: edit princip shem
Connections:
- net TX_Enable(Dynamixel_TTL) is gone; now on net TX_EN: D1.1 (1OE#), D1.7 (2OE), R3.1
- net USART4_RX(Dynamixel_TTL) is gone; now on net USART6_RX: D1.6 (1Y), R4.2
- net USART6_TX is gone; now on net Data: U1.129 (PG14)
- net D39 renamed TX_EN
Changed lines of the file:
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@@
 	)
 	(junction
-		(at 77.47 212.09)
+		(at 200.66 46.99)
 		(diameter 0)
 		(color 0 0 0 0)
 	)
 	(junction
-		(at 200.66 46.99)
+		(at 77.47 212.09)
 		(diameter 0)
 		(color 0 0 0 0)
@@
 	)
 	(junction
-		(at 81.28 217.17)
-		(diameter 0)
-		(color 0 0 0 0)
-	)
-	(junction
 		(at 229.87 59.69)
 		(diameter 0)
@@
 	)
 	(junction
+		(at 81.28 217.17)
+		(diameter 0)
+		(color 0 0 0 0)
+	)
+	(junction
 		(at 115.57 138.43)
 		(diameter 0)
@@
 	(wire
 		(pts
-			(xy 81.28 217.17) (xy 82.55 217.17)
+			(xy 81.28 217.17) (xy 83.82 217.17)
 		)
 		(stroke
@@
 	(wire
 		(pts
-			(xy 77.47 212.09) (xy 82.55 212.09)
+			(xy 77.47 212.09) (xy 83.82 212.09)
 		)
 		(stroke
@@
 		)
 	)
+	(global_label "USART6_RX"
+		(shape input)
+		(at 83.82 212.09 0)
+		(fields_autoplaced yes)
+		(effects
+			(font
+				(size 1.27 1.27)
+			)
+			(justify left)
+		)
+		(property "Intersheetrefs" "${INTERSHEET_REFS}"
+			(at 97.328 212.09 0)
+			(hide yes)
+			(show_name no)
+			(do_not_autoplace no)
+			(effects
+				(font
+					(size 1.27 1.27)
+				)
+				(justify left)
+			)
+		)
+	)
 	(global_label "D11"
 		(shape input)
@@
 		)
 	)
+	(global_label "USART6_TX"
+		(shape input)
+		(at 83.82 217.17 0)
+		(fields_autoplaced yes)
+		(effects
+			(font
+				(size 1.27 1.27)
+			)
+			(justify left)
+		)
+		(property "Intersheetrefs" "${INTERSHEET_REFS}"
+			(at 97.0256 217.17 0)
+			(hide yes)
+			(show_name no)
+			(do_not_autoplace no)
+			(effects
+				(font
+					(size 1.27 1.27)
+				)
+				(justify left)
+			)
+		)
+	)
 	(global_label "SDIO_D0"
 		(shape input)
@@
 		)
 	)
-	(global_label "USART4_RX(Dynamixel_TTL)"
-		(shape input)
-		(at 82.55 212.09 0)
-		(effects
-			(font
-				(size 1.27 1.27)
-			)
-			(justify left)
-		)
-		(property "Intersheetrefs" "${INTERSHEET_REFS}"
-			(at 82.55 212.09 0)
-			(hide yes)
-			(show_name no)
-			(do_not_autoplace no)
-			(effects
-				(font
-					(size 1.27 1.27)
-				)
-			)
-		)
-	)
 	(global_label "D28"
 		(shape input)
@@
 		)
 	)
-	(global_label "TX_Enable(Dynamixel_TTL)"
-		(shape input)
-		(at 83.82 207.01 0)
-		(fields_autoplaced yes)
-		(effects
-			(font
-				(size 1.27 1.27)
-			)
-			(justify left)
-		)
-		(property "Intersheetrefs" "${INTERSHEET_REFS}"
-			(at 111.5396 207.01 0)
-			(hide yes)
-			(show_name no)
-			(do_not_autoplace no)
-			(effects
-				(font
-					(size 1.27 1.27)
-				)
-				(justify left)
-			)
-		)
-	)
 	(global_label "SPI4_MISO"
 		(shape input)
@@
 		)
 	)
-	(global_label "D39"
+	(global_label "TX_EN"
 		(shape input)
 		(at 173.99 125.73 180)
@@
 		)
 		(property "Intersheetrefs" "${INTERSHEET_REFS}"
-			(at 167.3158 125.73 0)
+			(at 165.3806 125.73 0)
 			(hide yes)
 			(show_name no)
@@
 		)
 	)
-	(global_label "USART4_TX(Dynamixel_TTL)"
+	(global_label "USB_DM"
 		(shape input)
-		(at 82.55 217.17 0)
+		(at 300.99 102.87 0)
+		(fields_autoplaced yes)
 		(effects
 			(font
@@
 		)
 		(property "Intersheetrefs" "${INTERSHEET_REFS}"
-			(at 82.55 217.17 0)
+			(at 311.4742 102.87 0)
 			(hide yes)
 			(show_name no)
@@
 					(size 1.27 1.27)
 				)
+				(justify left)
 			)
 		)
 	)
-	(global_label "USB_DM"
+	(global_label "VREF+"
 		(shape input)
-		(at 300.99 102.87 0)
+		(at 173.99 85.09 180)
 		(fields_autoplaced yes)
 		(effects
@@
 				(size 1.27 1.27)
 			)
-			(justify left)
+			(justify right)
 		)
 		(property "Intersheetrefs" "${INTERSHEET_REFS}"
-			(at 311.4742 102.87 0)
+			(at 164.8362 85.09 0)
 			(hide yes)
 			(show_name no)
@@
 					(size 1.27 1.27)
 				)
-				(justify left)
+				(justify right)
 			)
 		)
 	)
-	(global_label "VREF+"
+	(global_label "TX_EN"
 		(shape input)
-		(at 173.99 85.09 180)
+		(at 83.82 207.01 0)
 		(fields_autoplaced yes)
 		(effects
@@
 				(size 1.27 1.27)
 			)
-			(justify right)
+			(justify left)
 		)
 		(property "Intersheetrefs" "${INTERSHEET_REFS}"
-			(at 164.8362 85.09 0)
+			(at 92.4294 207.01 0)
 			(hide yes)
 			(show_name no)
@@
 					(size 1.27 1.27)
 				)
-				(justify right)
+				(justify left)
 			)
 		)

Commit message: Very sad. Need new place
Parts:
- renumbered C7 to C10, C8 to C11, C10 to C12, C9 to C13, C11 to C14, C12 to C15, C13 to C16, C14 to C17, C15 to C18, C16 to C19, C17 to C20, C18 to C21, C19 to C22, C21 to C23, C32 to C24, C28 to C25, C24 to C26, C31 to C28, C34 to C29, C25 to C30, C26 to C31, C30 to C32, C5 to C4, C4 to C5, C20 to C6, C22 to C7, C23 to C8, C6 to C9, R2 to R1, R6 to R10, R25 to R13, R26 to R14, R27 to R15, R15 to R16, R16 to R17, R17 to R18, R18 to R19, R1 to R2, R19 to R20, R30 to R21, R31 to R22, R21 to R23, R22 to R24, R14 to R25, R13 to R26, R36 to R27, R33 to R28, R32 to R29, R5 to R3, R35 to R30, R37 to R31, R28 to R32, R29 to R33, R23 to R34, R24 to R35, R3 to R4, R8 to R5, R9 to R6, R4 to R7, R7 to R8, R10 to R9, SW2 to SW1, SW1 to SW2
