File: plat_logic.kicad_sch (KiCad schematic)
At the start: 80 parts, among them SW1 Button-SMD-4.5x4.5x5.5, SW2 Button-SMD-4.5x4.5x5.5, U1 STM32F429ZITx, U2 USBLC6-2SC6, Y1 CSTNE8M00GH5L000R0 8.000MHZ, Y2 NX3215SA-32.768KHZ-EXS00A-MU0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

Commit message: Дорожки
Other:
- moved on the sheet: R33
Changed lines of the file:
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@@
 	(wire
 		(pts
-			(xy 328.93 130.81) (xy 330.2 130.81)
+			(xy 321.31 130.81) (xy 330.2 130.81)
 		)
 		(stroke
@@
 	(wire
 		(pts
-			(xy 321.31 130.81) (xy 311.15 130.81)
+			(xy 313.69 130.81) (xy 311.15 130.81)
 		)
 		(stroke
@@
 	(symbol
 		(lib_id "Device:R")
-		(at 325.12 130.81 270)
+		(at 317.5 130.81 270)
 		(unit 1)
 		(body_style 1)
@@
 		(dnp no)
 		(property "Reference" "R33"
-			(at 330.962 128.778 90)
+			(at 315.722 133.096 90)
 			(show_name no)
 			(do_not_autoplace no)
@@
 		)
 		(property "Value" "2.2k"
-			(at 330.962 130.556 90)
+			(at 315.722 134.874 90)
 			(show_name no)
 			(do_not_autoplace no)
@@
 		)
 		(property "Footprint" "Resistor_SMD:R_0603_1608Metric"
-			(at 325.12 129.032 90)
+			(at 317.5 129.032 90)
 			(hide yes)
 			(show_name no)
@@
 		)
 		(property "Datasheet" ""
-			(at 325.12 130.81 0)
+			(at 317.5 130.81 0)
 			(hide yes)
 			(show_name no)
@@
 		)
 		(property "Description" "Resistor"
-			(at 325.12 130.81 0)
+			(at 317.5 130.81 0)
 			(hide yes)
 			(show_name no)

Commit message: final
Parts:
- removed C2, C3: 12pF, Capacitor_SMD:C_0603_1608Metric, symbol Device:C
- removed Y1: CSTNE8M00GH5L000R0 8.000MHZ, Crystal:Crystal_SMD_3215-2Pin_3.2x1.5mm, symbol Device:Crystal
- added Y3: CSTNE8M00GH5L000R0 8.000MHZ, Crystal:Resonator_SMD_Murata_CSTxExxV-3Pin_3.0x1.1mm, symbol Device:Crystal_GND2
Connections:
- net GND: now also Y3.2
- net PH0: now also Y3.1
- net at R8.2: now also Y3.3

Commit message: Iter2
Connections:
- net D33 is gone; now on net D27: U1.90 (PG5)
- net D34 is gone; now on net D28: U1.91 (PG6)
- net D35 is gone; now on net D29: U1.110 (PA15)
- net D36 is gone; now on net D30: U1.119 (PD5)
- net D37 is gone; now on net D31: U1.123 (PD7)
- net D38 is gone; now on net D32: U1.125 (PG10)
- net D10: now also U1.50 (PF12); no longer U1.27 (PC1)
- net D11: now also U1.53 (PF13); no longer U1.37 (PA3)
- net D12: now also U1.54 (PF14); no longer U1.49 (PF11)
- net D13: now also U1.55 (PF15); no longer U1.50 (PF12)
- net D14: now also U1.56 (PG0); no longer U1.53 (PF13)
- net D15: now also U1.57 (PG1); no longer U1.54 (PF14)
- net D16: now also U1.63 (PE10); no longer U1.55 (PF15)
- net D17: now also U1.73 (PB12); no longer U1.56 (PG0)
- net D18: now also U1.79 (PD10); no longer U1.57 (PG1)
- net D19: now also U1.80 (PD11); no longer U1.58 (PE7)
- net D20: now also U1.81 (PD12); no longer U1.59 (PE8)
- net D21: now also U1.82 (PD13); no longer U1.63 (PE10)
- net D22: now also U1.85 (PD14); no longer U1.73 (PB12)
- net D23: now also U1.86 (PD15); no longer U1.74 (PB13)
- net D24: now also U1.87 (PG2); no longer U1.79 (PD10)
- net D25: now also U1.88 (PG3); no longer U1.80 (PD11)
- net D26: now also U1.89 (PG4); no longer U1.81 (PD12)
- net D27: no longer U1.82 (PD13)
- net D28: no longer U1.85 (PD14)
- net D29: no longer U1.86 (PD15)
- net D3: now also U1.7 (PC13); no longer U1.4 (PE5)
- net D30: no longer U1.87 (PG2)
- net D31: no longer U1.88 (PG3)
- net D32: no longer U1.89 (PG4)
- net D4: now also U1.12 (PF2); no longer U1.5 (PE6)
- net D5: now also U1.22 (PF10); no longer U1.7 (PC13)
- net D6: now also U1.26 (PC0); no longer U1.12 (PF2)
- net D7: now also U1.27 (PC1); no longer U1.21 (PF9)
- net D8: now also U1.37 (PA3); no longer U1.22 (PF10)
- net D9: now also U1.49 (PF11); no longer U1.26 (PC0)
- net FS4: now also U1.21 (PF9); no longer U1.18 (PF6)
- net IN1_M1: now also U1.4 (PE5); no longer U1.75 (PB14)
- net IN1_M2: now also U1.5 (PE6); no longer U1.76 (PB15)
- net at U1.103 (PA11): now also U2.3 (I/O2); no longer U2.1 (I/O1)
- net at U1.104 (PA12): now also U2.1 (I/O1); no longer U2.3 (I/O2)
- new net PWM_ard: U1.18 (PF6)
- new net SPI2_MISO: U1.75 (PB14)
- new net SPI2_MOSI: U1.76 (PB15)
- new net SPI2_SCK: U1.74 (PB13)
- new net UART7_RX: U1.58 (PE7)
- new net UART7_TX: U1.59 (PE8)
Other:
- note added: "UART7 SPI2 Идут на ардуину"
- moved on the sheet: U2

Commit message: Trass
Parts:
- renumbered C12 to C10, C13 to C11, C14 to C12, C15 to C13, C16 to C14, C17 to C15, C18 to C16, C19 to C17, C20 to C18, C21 to C19, C4 to C2, C22 to C20, C23 to C21, C24 to C22, C25 to C23, C26 to C24, C27 to C25, C28 to C26, C29 to C27, C30 to C28, C31 to C29, C5 to C3, C32 to C30, C33 to C31, C6 to C4, C7 to C5, C8 to C6, C9 to C7, C10 to C8, C11 to C9, Y3 to Y1
Other:
- note added: "UART7 SPI2 I2C2 Идут на ардуину"
- note removed: "UART7 SPI2 Идут на ардуину"
