File: plat_logic.kicad_pcb (KiCad board)
At the start: 2 copper layers, 137 parts, among them CN1 GPS_Port, CN2 SM06B-GHS-TB(LF)(SN), Con2 DS1023-1X2SF11, Con3 DS1023-1X10SF11, Con4 DS1023-1X6SF11, J1 USB_C_Receptacle, J10 DS1023-1X5SF11, J11 DS1023-1X5SF11, J12 DS1023-1X5SF11, J13 DS1023-1X5SF11, J14 DS1023-1X5SF11, J2 DS1023-1X9S21, J3 DS1023-1X7SF11, J4 DS1023-1X8SF11, J5 DS1023-1X6SF11, J6 DS1023-1X6SF11, J7 DS1023-1X8SF11, J8 DS1023-1X8SF11, J9 DS1023-1X5SF11, SW1 Button-SMD-4.5x4.5x5.5, SW2 Button-SMD-4.5x4.5x5.5, U1 STM32F429ZITx, U2 USBLC6-2SC6, U3 FT232RL, Y1 NX3225GD 8.000MHZ EXS00A-CG06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, Y2 NX3215SA-32.768KHZ-EXS00A-MU0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, con1 DS1023-1X3SF11

Commit message: На компе сделать
Parts:
- moved Con4 112.8 mm to (167.6, 48.4), turned to -90 degrees
- moved C4 37.7 mm to (154.5, 51.0)
- moved SW1 31.4 mm to (153.3, 55.5), turned to 90 degrees
- moved D2 30.8 mm to (150.6, 50.2)
- moved R10 30.8 mm to (152.2, 50.2)
- moved R26 13.6 mm to (137.4, 85.1)
- moved R27 11.8 mm to (134.9, 87.2)
- moved C22 11.4 mm to (134.2, 85.3), turned to 180 degrees
- moved D5 11.1 mm to (160.0, 38.6)
- moved D6 11.1 mm to (158.0, 38.6)
- moved R53 11.1 mm to (158.0, 41.9)
- moved R52 11.1 mm to (160.0, 41.9)
- moved R25 11.1 mm to (137.4, 83.1)
- moved C23 10.1 mm to (131.6, 87.5), turned to 180 degrees
- moved C20 8.07 mm to (134.2, 83.3), turned to 0 degrees
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Routing:
- net NRST: track 6.87 -> 47.8 mm, vias 0 -> 2
- net Net-(U1-PC1): track 0.00 -> 10.6 mm, vias 0 -> 2
- net Net-(U1-PC0): track 0.00 -> 9.80 mm, vias 0 -> 2
- net GND: track 8.05 -> 12.1 mm
- net IN1_M5: track 0.00 -> 1.36 mm, vias 0 -> 1
- net IN1_M6: track 0.00 -> 1.26 mm, vias 0 -> 1
- net Net-(U1-PC2): track 0.00 -> 1.22 mm, vias 0 -> 1
- net Net-(U1-PC3): track 0.00 -> 1.20 mm, vias 0 -> 1

Commit message: edit princip shem
Parts:
- removed C29: 100nF, Capacitor_SMD:C_0603_1608Metric
- removed C35: 22pF, Capacitor_SMD:C_0603_1608Metric
- removed C37, C38: 0.1uF, Capacitor_SMD:C_0603_1608Metric
- removed C39: 10uF, Capacitor_SMD:C_0603_1608Metric
- removed CN2: SM06B-GHS-TB(LF)(SN), Connector_JST:JST_GH_SM06B-GHS-TB_1x06-1MP_P1.25mm_Horizontal
- removed Con3: DS1023-1X10SF11, Connector_PinHeader_2.54mm:PinHeader_1x10_P2.54mm_Vertical
- removed D3: red, LED_SMD:LED_0603_1608Metric
- removed D4: green, LED_SMD:LED_0603_1608Metric
- removed F1: Polyfuse, Fuse:Fuse_0603_1608Metric
- removed F2: 04000025WR, Fuse:Fuse_0603_1608Metric
- removed J7, J8: DS1023-1X8SF11, Connector_PinHeader_2.54mm:PinHeader_1x08_P2.54mm_Vertical
- removed R48, R49: 330, Resistor_SMD:R_0805_2012Metric
- removed USB1: MICROUSB-5PIN, Connector_USB:USB_Micro-B_GCT_USB3076-30-A
- added C42: 100nF, Capacitor_SMD:C_0603_1608Metric, F.Cu at (214.3, 105.5)
- added C43: 1uF, Capacitor_SMD:C_0603_1608Metric, F.Cu at (214.3, 108.0)
- added C44: 100nF, Capacitor_SMD:C_0603_1608Metric, F.Cu at (214.3, 110.5)
- added D7: led, LED_SMD:LED_0603_1608Metric, F.Cu at (214.4, 116.6)
- added I2C2_conn3: SM04B-GHS-TB(LF)(SN), Connector_JST:JST_GH_SM04B-GHS-TB_1x04-1MP_P1.25mm_Horizontal, F.Cu at (144.5, 43.1)
- added I2C2_conn4: SM04B-GHS-TB(LF)(SN), Connector_JST:JST_GH_SM04B-GHS-TB_1x04-1MP_P1.25mm_Horizontal, F.Cu at (203.4, 89.9)
- added JP3: Jumper_2_Open, Jumper:SolderJumper-2_P1.3mm_Open_Pad1.0x1.5mm, F.Cu at (214.5, 113.5)
- added R54: 330, Resistor_SMD:R_0805_2012Metric, F.Cu at (210.1, 105.7)
- added R55: 1K5, Resistor_SMD:R_0805_2012Metric, F.Cu at (210.1, 108.6)
- added R56: 1K5, Resistor_SMD:R_0805_2012Metric, F.Cu at (210.1, 111.6)
- added XL1: JST_GH_SM06B-GHS-TB, Connector_JST:JST_GH_SM05B-GHS-TB_1x05-1MP_P1.25mm_Horizontal, F.Cu at (172.1, 41.2)
- added XL2: JST_GH_SM06B-GHS-TB, Connector_JST:JST_GH_SM05B-GHS-TB_1x05-1MP_P1.25mm_Horizontal, F.Cu at (164.2, 108.5)
- added XL3: JST_GH_SM06B-GHS-TB, Connector_JST:JST_GH_SM05B-GHS-TB_1x05-1MP_P1.25mm_Horizontal, F.Cu at (152.1, 109.0)
- added XL4: JST_GH_SM06B-GHS-TB, Connector_JST:JST_GH_SM05B-GHS-TB_1x05-1MP_P1.25mm_Horizontal, F.Cu at (177.4, 56.3)
- Con4: value DS1023-1X6SF11 -> DS1023-1X5SF11; footprint Connector_PinHeader_2.54mm:PinHeader_1x06_P2.54mm_Vertical -> Connector_PinHeader_2.54mm:PinHeader_1x05_P2.54mm_Vertical
- J1: footprint Connector_USB:USB_C_Receptacle_JAE_DX07S024WJ1R350 -> Connector_USB:USB_C_Receptacle_HRO_TYPE-C-31-M-12
- J2: value DS1023-1X9S21 -> DS1023-1X6SF11; footprint Connector_PinHeader_2.54mm:PinHeader_1x09_P2.54mm_Vertical -> Connector_PinHeader_2.54mm:PinHeader_1x06_P2.54mm_Vertical
- J3: value DS1023-1X7SF11 -> DS1023-1X8SF11; footprint Connector_PinHeader_2.54mm:PinHeader_1x07_P2.54mm_Vertical -> Connector_PinHeader_2.54mm:PinHeader_1x08_P2.54mm_Vertical
- J4: value DS1023-1X8SF11 -> DS1023-1X11S21; footprint Connector_PinHeader_2.54mm:PinHeader_1x08_P2.54mm_Vertical -> Connector_PinHeader_2.54mm:PinHeader_1x11_P2.54mm_Vertical
- J5, J6: value DS1023-1X6SF11 -> DS1023-1X11S21; footprint Connector_PinHeader_2.54mm:PinHeader_1x06_P2.54mm_Vertical -> Connector_PinHeader_2.54mm:PinHeader_1x11_P2.54mm_Vertical
- R20: value 1k -> 10k
- R34: value 47 -> 10k; footprint Resistor_SMD:R_0805_2012Metric -> Resistor_SMD:R_0603_1608Metric
- R38: value 27K -> 120; footprint Resistor_SMD:R_0805_2012Metric -> Resistor_SMD:R_0603_1608Metric
- R6: value 0 -> 1М
- R7: value 100K -> 330
- U3: value FT232RL -> SN65HVD232; footprint Package_SO:SSOP-28_5.3x10.2mm_P0.65mm -> Package_SO:SOIC-8_3.9x4.9mm_P1.27mm
- Y1: value NX3225GD 8.000MHZ EXS00A-CG06684 -> CSTNE8M00GH5L000R0 8.000MHZ; footprint Crystal:Crystal_SMD_3225-4Pin_3.2x2.5mm -> Crystal:Crystal_SMD_3215-2Pin_3.2x1.5mm
- moved J4 9.62 mm to (90.2, 125.3)
Connections:
- C10 pad 2: Net-(C10-Pad2) -> GND
- C11 pad 1: +3v3 -> GND
- C11 pad 2: Net-(C11-Pad2) -> +3v3
- C12 pad 2: Net-(C12-Pad2) -> GND
- C13 pad 1: +3v3 -> GND
- C13 pad 2: Net-(C13-Pad2) -> +3v3
- C14 pad 1: +3v3 -> GND
- C14 pad 2: Net-(C14-Pad2) -> +3v3
- C15 pad 1: +3v3 -> GND
- C15 pad 2: Net-(C15-Pad2) -> +3v3
- C16 pad 1: +3v3 -> GND
- C16 pad 2: Net-(C16-Pad2) -> +3v3
- C17 pad 1: +3v3 -> GND
- C17 pad 2: Net-(C17-Pad2) -> +3v3
- C18 pad 1: +3v3 -> GND
- C18 pad 2: Net-(C18-Pad2) -> +3v3
- C19 pad 1: +3v3 -> GND
- C19 pad 2: Net-(C19-Pad2) -> +3v3
- C2 pad 2: Net-(C2-Pad2) -> PH0
- C21 pad 1: +3v3 -> GND
- C21 pad 2: Net-(C21-Pad2) -> +3v3
- C24 pad 1: +3v3 -> GND
- C24 pad 2: Net-(C24-Pad2) -> +3v3
- C27 pad 1: A3 -> GND
- C27 pad 2: GND -> A3
- C34 pad 1: DAC(PA4) -> DAC
- C40 pad 1: VBUS(PA9) -> +5v
- C41 pad 1: VBUS(PA9) -> +5v
- CN1 pad 1: VBUS(PA9) -> +5v
- CN1 pad 2: USART7_TX -> USART1_TX
- CN1 pad 3: USART7_RX -> USART1_RX
- Con2 pad 1: I2C_SCL -> I2C3_SCL
- Con2 pad 2: I2C_SDA -> I2C3_SDA
- Con4 pad 1: GND -> +3v3
- Con4 pad 2: JTDI -> NRST
- Con4 pad 3: CLK -> SWDIO
- Con4 pad 4: SWDIO -> CLK
- Con4 pad 5: NRST -> GND
- D1 pad 1: TX_Enable(Dynamixel_TTL) -> TX_EN
- D1 pad 5: USART4_TX(Dynamixel_TTL) -> Data
- D1 pad 6: USART4_RX(Dynamixel_TTL) -> USART6_RX
- D1 pad 7: TX_Enable(Dynamixel_TTL) -> TX_EN
- DynamixelCon1 pad 2: VBUS(PA9) -> +5v
- I2C2_conn2 pad 2: I2C_SCL -> I2C2_SLC
- I2C2_conn2 pad 3: I2C_SDA -> I2C2_SDA
- J1 pad A4: Net-(F1-Pad2) -> unconnected-(J1-VBUS-PadA4)
- J1 pad A6: USBDP(PA11) -> USB_DP
- J1 pad A7: USBDM(PA12) -> USB_DM
- J1 pad A9: Net-(F1-Pad2) -> unconnected-(J1-VBUS-PadA4)_2
- J1 pad B4: Net-(F1-Pad2) -> unconnected-(J1-VBUS-PadA4)_1
- J1 pad B6: USBDP(PA11) -> USB_DP
- J1 pad B7: USBDM(PA12) -> USB_DM
- J1 pad B9: Net-(F1-Pad2) -> unconnected-(J1-VBUS-PadA4)_3
- J2 pad 1: D0 -> D33
- J2 pad 2: D1 -> D34
- J2 pad 3: D2 -> D35
- J2 pad 4: D3 -> D36
- J2 pad 5: D4 -> D37
- J2 pad 6: D5 -> D38
- J3 pad 1: D37 -> A0
- J3 pad 2: D38 -> A1
- J3 pad 3: D39 -> A2
- J3 pad 4: D40 -> A3
- J3 pad 5: D41 -> A4
- J3 pad 6: D42 -> A5
- J3 pad 7: D43 -> A6
- J4 pad 1: D44 -> D0
- J4 pad 2: D45 -> D1
- J4 pad 3: D46 -> D2
- J4 pad 4: D47 -> D3
- J4 pad 5: D48 -> D4
- J4 pad 6: D49 -> D5
- J4 pad 7: D50 -> D6
- J4 pad 8: D51 -> D7
- J5 pad 1: D9 -> D11
- J5 pad 2: D10 -> D12
- J5 pad 3: D11 -> D13
- J5 pad 4: D12 -> D14
- J5 pad 5: D13 -> D15
- J5 pad 6: D14 -> D16
- J6 pad 1: D15 -> D22
- J6 pad 2: D16 -> D23
- J6 pad 3: D17 -> D24
- J6 pad 4: D18 -> D25
- J6 pad 5: D19 -> D26
- J6 pad 6: D20 -> D27
- R13 pad 2: ENC_A_M1_mk -> ENC_B_M1_mk
- R14 pad 1: ENC_B_M1_mk -> ENC_A_M1_mk
- R20 pad 1: Net-(U1-PA9) -> +3v3
- R20 pad 2: VBUS(PA9) -> SDIO_CMD
- R25 pad 2: Net-(U1-PC0) -> Net-(U1-PF3)
- R26 pad 2: Net-(U1-PC1) -> Net-(U1-PF4)
- R27 pad 2: Net-(U1-PC2) -> Net-(U1-PF5)
- R3 pad 1: TX_Enable(Dynamixel_TTL) -> TX_EN
- R32 pad 2: Net-(U1-PC3) -> Net-(U1-PC4)
- R33 pad 2: Net-(U1-PA2) -> Net-(U1-PB1)
- R34 pad 1: A7 -> +3v3
- R34 pad 2: Net-(U1-PA3) -> SDIO_D0
- R35 pad 2: Net-(U1-PC4) -> Net-(U1-PC5)
- R36 pad 2: Net-(U1-PC5) -> Net-(U1-PB0)
- R37 pad 1: DAC(PA4) -> DAC
- R38 pad 1: DAC(PA5) -> Net-(U3-CANH)
- R38 pad 2: GND -> Net-(JP3-A)
- R4 pad 2: USART4_RX(Dynamixel_TTL) -> USART6_RX
- R42 pad 2: I2C_SCL -> I2C1_SCL
- R43 pad 2: I2C_SDA -> I2C1_SDA
- R44 pad 2: I2C_SCL -> I2C1_SCL
- R45 pad 2: I2C_SCL -> I2C1_SCL
- R46 pad 2: I2C_SDA -> I2C1_SDA
- R47 pad 2: I2C_SDA -> I2C1_SDA
- R50 pad 2: I2C_SCL -> I2C2_SLC
- R51 pad 2: I2C_SDA -> I2C2_SDA
- R52 pad 1: D49 -> D37
- R53 pad 1: D48 -> D38
- R6 pad 2: Net-(C2-Pad2) -> PH1
- U1 pad 10: I2C_SDA -> I2C2_SDA
- U1 pad 100: D35 -> I2C3_SCL
- U1 pad 101: Net-(U1-PA9) -> USART1_TX
- U1 pad 102: D36 -> USART1_RX
- U1 pad 108: Net-(C18-Pad2) -> +3v3
- U1 pad 11: I2C_SCL -> I2C2_SLC
- U1 pad 110: JTDI -> D35
- U1 pad 111: USART4_TX(Dynamixel_TTL) -> SPI3_SCK
- U1 pad 112: USART4_RX(Dynamixel_TTL) -> SPI3_MISO
- U1 pad 113: TX_Enable(Dynamixel_TTL) -> SDIO_CK
- U1 pad 114: D37 -> CAN1_RX
- U1 pad 115: D38 -> CAN1_TX
- U1 pad 116: D39 -> SDIO_CMD
- U1 pad 117: D40 -> ENC_A_M2_mk
- U1 pad 118: D41 -> ENC_B_M2_mk
- U1 pad 119: D42 -> D36
- U1 pad 12: D4 -> D6
- U1 pad 121: Net-(C19-Pad2) -> +3v3
- U1 pad 122: D43 -> SPI3_MOSI
- U1 pad 123: D44 -> D37
- U1 pad 124: D45 -> USART6_RX
- U1 pad 125: D46 -> D38
- U1 pad 126: D47 -> TX_EN
- U1 pad 128: D48 -> IN2_M3
- U1 pad 129: D49 -> Data
- U1 pad 13: D5 -> Net-(U1-PF3)
- U1 pad 131: Net-(C21-Pad2) -> +3v3
- U1 pad 132: D50 -> FS3
- U1 pad 133: SWO -> IN1_M3
- U1 pad 134: D51 -> ENC_A_M3_mk
- U1 pad 135: IN2_M3 -> ENC_B_M3_mk
- U1 pad 136: IN2_M4 -> ENC_A_M4_mk
- U1 pad 137: IN2_M5 -> ENC_B_M4_mk
- U1 pad 139: IN2_M6 -> I2C1_SCL
- U1 pad 14: D6 -> Net-(U1-PF4)
- U1 pad 140: FS1 -> I2C1_SDA
- U1 pad 144: Net-(C24-Pad2) -> +3v3
- U1 pad 15: D7 -> Net-(U1-PF5)
- U1 pad 17: Net-(C10-Pad2) -> +3v3
- U1 pad 18: IN1_M3 -> FS4
- U1 pad 20: IN1_M5 -> IN2_M4
- U1 pad 21: IN1_M6 -> D7
- U1 pad 26: Net-(U1-PC0) -> D9
- U1 pad 27: Net-(U1-PC1) -> D10
- U1 pad 28: Net-(U1-PC2) -> FS5
- U1 pad 29: Net-(U1-PC3) -> IN2_M5
- U1 pad 30: Net-(C11-Pad2) -> +3v3
- U1 pad 34: ENC_A_M2_mk -> ENC_A_M5_mk
- U1 pad 35: ENC_B_M2_mk -> ENC_B_M5_mk
- U1 pad 36: Net-(U1-PA2) -> IN1_M5
- U1 pad 37: Net-(U1-PA3) -> D11
- U1 pad 39: Net-(C12-Pad2) -> +3v3
- U1 pad 4: ENC_A_M6_mk -> D3
- U1 pad 40: DAC(PA4) -> DAC
- U1 pad 41: DAC(PA5) -> SPI1_SCK
- U1 pad 42: ENC_A_M3_mk -> SPI1_MISO
- U1 pad 43: ENC_B_M3_mk -> SPI1_MOSI
- U1 pad 46: IN2_M1 -> Net-(U1-PB0)
- U1 pad 47: IN2_M2 -> Net-(U1-PB1)
- U1 pad 49: D9 -> D12
- U1 pad 5: ENC_B_M6_mk -> D4
- U1 pad 50: D10 -> D13
- U1 pad 52: Net-(C13-Pad2) -> +3v3
- U1 pad 53: D11 -> D14
- U1 pad 54: D12 -> D15
- U1 pad 55: D13 -> D16
- U1 pad 56: D14 -> D17
- U1 pad 57: D15 -> D18
- U1 pad 58: USART7_RX -> D19
- U1 pad 59: USART7_TX -> D20
- U1 pad 60: ENC_A_M1_mk -> ENC_A_M6_mk
- U1 pad 62: Net-(C14-Pad2) -> +3v3
- U1 pad 63: D16 -> D21
- U1 pad 64: ENC_B_M1_mk -> ENC_B_M6_mk
- U1 pad 65: D17 -> SPI4_SCK
- U1 pad 66: D18 -> SPI4_MISO
- U1 pad 67: D19 -> SPI4_MOSI
- U1 pad 68: D20 -> FS6
- U1 pad 69: FS2 -> IN2_M6
- U1 pad 7: D3 -> D5
- U1 pad 70: FS3 -> IN1_M6
- U1 pad 72: Net-(C15-Pad2) -> +3v3
- U1 pad 73: FS4 -> D22
- U1 pad 74: FS5 -> D23
- U1 pad 77: FS6 -> IN2_M2
- U1 pad 78: D21 -> FS2
- U1 pad 79: D22 -> D24
- U1 pad 80: D23 -> D25
- U1 pad 81: ENC_A_M4_mk -> D26
- U1 pad 82: ENC_B_M4_mk -> D27
- U1 pad 84: Net-(C16-Pad2) -> +3v3
- U1 pad 85: D24 -> D28
- U1 pad 86: D25 -> D29
- U1 pad 87: D26 -> D30
- U1 pad 88: D27 -> D31
- U1 pad 89: D28 -> D32
- U1 pad 90: D29 -> D33
- U1 pad 91: D30 -> D34
- U1 pad 92: D31 -> IN2_M1
- U1 pad 93: D32 -> FS1
- U1 pad 95: Net-(C17-Pad2) -> +3v3
- U1 pad 96: ENC_A_M5_mk -> ENC_A_M1_mk
- U1 pad 97: ENC_B_M5_mk -> ENC_B_M1_mk
- U1 pad 98: D33 -> SDIO_D0
- U1 pad 99: D34 -> I2C3_SDA
- U2 pad 1: Net-(U1-PA12) -> Net-(U1-PA11)
- U2 pad 3: Net-(U1-PA11) -> Net-(U1-PA12)
- U2 pad 4: USBDP(PA11) -> USB_DM
- U2 pad 5: VBUS(PA9) -> +5v
- U2 pad 6: USBDM(PA12) -> USB_DP
- U3 pad 1: UART8_TX -> CAN1_TX
- U3 pad 2: unconnected-(U3-DTR#-Pad2) -> GND
- U3 pad 3: unconnected-(U3-RTS#-Pad3) -> +3v3
- U3 pad 4: +3v3 -> CAN1_RX
- U3 pad 5: UART8_RX -> unconnected-(U3-NC-Pad5)
- U3 pad 6: unconnected-(U3-RI#-Pad6) -> Net-(JP3-B)
- U3 pad 7: GND -> Net-(U3-CANH)
- Y1 pad 2: Net-(C2-Pad2) -> PH0
- con1 pad 2: VBUS(PA9) -> +5v
Routing:
- net NRST: track 47.8 -> 19.1 mm, vias 2 -> 0
- net +3v3: track 1.62 -> 14.8 mm
- net Net-(U1-PC1): track 10.6 -> 0.00 mm, vias 2 -> 0
- net Net-(U1-PC0): track 9.80 -> 0.00 mm, vias 2 -> 0
- net Net-(C10-Pad2): track 4.91 -> 0.00 mm
- net ENC_A_M1_mk: track 5.18 -> 0.27 mm
- net Net-(C11-Pad2): track 4.87 -> 0.00 mm
- net ENC_B_M1_mk: track 5.17 -> 0.30 mm
- net Net-(C2-Pad2): track 4.51 -> 0.00 mm
- net (no net): track 2.20 -> 6.71 mm
- net Net-(C17-Pad2): track 2.31 -> 0.00 mm
- net Net-(C19-Pad2): track 2.22 -> 0.00 mm
- net Net-(C21-Pad2): track 2.19 -> 0.00 mm
- net Net-(C16-Pad2): track 2.17 -> 0.00 mm
- net Net-(C14-Pad2): track 2.09 -> 0.00 mm
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
Commit message: Very sad. Need new place
Parts:
- removed C40: C_Polarized_US, Capacitor_SMD:C_0603_1608Metric
- removed C41: 0.1uF, Capacitor_SMD:C_0603_1608Metric
- removed C42, C44: 100nF, Capacitor_SMD:C_0603_1608Metric
- removed C43: 1uF, Capacitor_SMD:C_0603_1608Metric
- removed Con4: DS1023-1X5SF11, Connector_PinHeader_2.54mm:PinHeader_1x05_P2.54mm_Vertical
- removed D6, D7: led, LED_SMD:LED_0603_1608Metric
- removed R55, R56: 1K5, Resistor_SMD:R_0805_2012Metric
- removed XL1, XL2, XL3, XL4: JST_GH_SM06B-GHS-TB, Connector_JST:JST_GH_SM05B-GHS-TB_1x05-1MP_P1.25mm_Horizontal
- added C29: 22pF, Capacitor_SMD:C_0603_1608Metric, F.Cu at (224.9, 68.8)
- added C35: 100nF, Capacitor_SMD:C_0603_1608Metric, F.Cu at (224.9, 83.8)
- added C37: 0.1uF, Capacitor_SMD:C_0603_1608Metric, F.Cu at (228.9, 66.2)
- added C38: 100nF, Capacitor_SMD:C_0603_1608Metric, F.Cu at (228.9, 68.8)
- added C39: 1uF, Capacitor_SMD:C_0603_1608Metric, F.Cu at (228.9, 71.3)
- added D3: led, LED_SMD:LED_0603_1608Metric, F.Cu at (241.6, 132.8)
- added D4: led, LED_SMD:LED_0603_1608Metric, F.Cu at (241.6, 135.3)
- added J15: DS1023-1X5SF11, Connector_PinHeader_2.54mm:PinHeader_1x05_P2.54mm_Vertical, F.Cu at (255.9, 89.9)
- added J16: DS1023-1X5SF11, Connector_PinHeader_2.54mm:PinHeader_1x05_P2.54mm_Vertical, F.Cu at (260.5, 89.9)
- added J17: DS1023-1X5SF11, Connector_PinHeader_2.54mm:PinHeader_1x05_P2.54mm_Vertical, F.Cu at (265.1, 89.9)
- added J7: DS1023-1X11S21, Connector_PinHeader_2.54mm:PinHeader_1x11_P2.54mm_Vertical, F.Cu at (259.8, 104.6)
- added J8: DS1023-1X6SF11, Connector_PinHeader_2.54mm:PinHeader_1x06_P2.54mm_Vertical, F.Cu at (257.5, 67.3)
- added R48: 1K5, Resistor_SMD:R_0805_2012Metric, F.Cu at (246.3, 127.4)
- added R49: 1K5, Resistor_SMD:R_0805_2012Metric, F.Cu at (250.7, 103.8)
- C11: value 100nF -> 1uF x5r
- C25, C26: value 12pF -> 100nF
- C30, C31: value 100nF -> 12pF
- C34: value 22pF -> 0.01uF
- C36: value 0.01uF -> C_Polarized_US
- C8: value 1uF x5r -> 100nF
- J10: value DS1023-1X5SF11 -> DS1023-1X8SF11; footprint Connector_PinHeader_2.54mm:PinHeader_1x05_P2.54mm_Vertical -> Connector_PinHeader_2.54mm:PinHeader_1x08_P2.54mm_Vertical
- J2: value DS1023-1X6SF11 -> JST_GH_SM06B-GHS-TB; footprint Connector_PinHeader_2.54mm:PinHeader_1x06_P2.54mm_Vertical -> Connector_JST:JST_GH_SM05B-GHS-TB_1x05-1MP_P1.25mm_Horizontal
- J3: value DS1023-1X8SF11 -> JST_GH_SM06B-GHS-TB; footprint Connector_PinHeader_2.54mm:PinHeader_1x08_P2.54mm_Vertical -> Connector_JST:JST_GH_SM05B-GHS-TB_1x05-1MP_P1.25mm_Horizontal
- J4, J5: value DS1023-1X11S21 -> JST_GH_SM06B-GHS-TB; footprint Connector_PinHeader_2.54mm:PinHeader_1x11_P2.54mm_Vertical -> Connector_JST:JST_GH_SM05B-GHS-TB_1x05-1MP_P1.25mm_Horizontal
- J9: value DS1023-1X5SF11 -> DS1023-1X11S21; footprint Connector_PinHeader_2.54mm:PinHeader_1x05_P2.54mm_Vertical -> Connector_PinHeader_2.54mm:PinHeader_1x11_P2.54mm_Vertical
- R1: value 10k -> 10K
- R10: value 10K -> 1М; footprint Resistor_SMD:R_0603_1608Metric -> Resistor_SMD:R_0805_2012Metric
- R13, R14, R15, R28, R29, R30: value 2.2k -> 47; footprint Resistor_SMD:R_0603_1608Metric -> Resistor_SMD:R_0805_2012Metric
- R17: value 0 -> 2.2k; footprint Resistor_SMD:R_0805_2012Metric -> Resistor_SMD:R_0603_1608Metric
- R2: value 10K -> 10k
- R20: value 10k -> 0; footprint Resistor_SMD:R_0603_1608Metric -> Resistor_SMD:R_0805_2012Metric
- R25, R26, R32, R33, R35: value 47 -> 2.2k; footprint Resistor_SMD:R_0805_2012Metric -> Resistor_SMD:R_0603_1608Metric
- R3: value 10k -> 100K; footprint Resistor_SMD:R_0603_1608Metric -> Resistor_SMD:R_0805_2012Metric
- R31: value 2.2k -> 27K; footprint Resistor_SMD:R_0603_1608Metric -> Resistor_SMD:R_0805_2012Metric
- R34: value 10k -> 2.2k
- R36: value 47 -> 1M
- R37: value 27K -> 6.8k
- R38: value 120 -> 6.8k; footprint Resistor_SMD:R_0603_1608Metric -> Resistor_SMD:R_0805_2012Metric
- R39: value 1M -> 10k; footprint Resistor_SMD:R_0805_2012Metric -> Resistor_SMD:R_0603_1608Metric
- R40: value 6.8k -> 10k; footprint Resistor_SMD:R_0805_2012Metric -> Resistor_SMD:R_0603_1608Metric
- R41: value 6.8k -> 1K5
- R43: value 1K5 -> 120; footprint Resistor_SMD:R_0805_2012Metric -> Resistor_SMD:R_0603_1608Metric
- R5: value 100K -> 0
- R50, R51: value 1K5 -> 100
- R52: value 100 -> 330
- R53: value 100 -> 1K5
- R54: value 330 -> 1K5
- R6: value 1М -> 10K; footprint Resistor_SMD:R_0805_2012Metric -> Resistor_SMD:R_0603_1608Metric
- R7: value 330 -> 10k; footprint Resistor_SMD:R_0805_2012Metric -> Resistor_SMD:R_0603_1608Metric
- R8: value 0 -> 330
- moved Con2 161.9 mm to (268.2, 134.6)
- moved CN1 159.1 mm to (259.4, 136.0), turned to 0 degrees
- moved J6 157.5 mm to (255.2, 104.6)
- moved R50 140.8 mm to (250.7, 106.8), turned to 0 degrees
- moved R51 140.6 mm to (250.7, 109.7), turned to 0 degrees
- moved R46 135.3 mm to (246.3, 121.5), turned to 0 degrees
- moved R47 133.6 mm to (246.3, 124.5)
- moved R45 132.5 mm to (246.3, 118.5)
- moved I2C2_conn2 129.9 mm to (227.9, 123.1), turned to 0 degrees
- moved R44 129.7 mm to (246.3, 115.6), turned to 0 degrees
- moved D5 128.6 mm to (241.6, 137.9), turned to 0 degrees
- moved R42 126.9 mm to (246.3, 112.7), turned to 0 degrees
- moved J4 126.7 mm to (216.8, 130.6)
- moved J5 122.9 mm to (216.8, 138.0)
- moved D2 121.1 mm to (241.6, 130.2), turned to 0 degrees
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Connections:
- C10 pad 1: +3v3 -> GND
- C10 pad 2: GND -> Net-(C10-Pad2)
- C11 pad 2: +3v3 -> Net-(C11-Pad2)
- C13 pad 1: GND -> Net-(C11-Pad2)
- C13 pad 2: +3v3 -> Net-(U1-VBAT)
- C15 pad 1: GND -> +3v3
- C15 pad 2: +3v3 -> GND
- C20 pad 2: A0 -> +3v3
- C22 pad 1: A1 -> GND
- C22 pad 2: GND -> +3v3
- C23 pad 1: A2 -> GND
- C23 pad 2: GND -> +3v3
- C24 pad 2: +3v3 -> A5
- C25 pad 1: PC15 -> A6
- C26 pad 1: PC14 -> GND
- C26 pad 2: GND -> +3v3
- C28 pad 1: A6 -> A4
- C30 pad 1: VDDA -> PC15
- C30 pad 2: VREF+ -> GND
- C31 pad 1: A4 -> PC14
- C32 pad 1: GND -> VDDA
- C32 pad 2: A5 -> VREF+
- C34 pad 1: DAC -> Net-(J1-SHIELD)
- C36 pad 1: Net-(J1-SHIELD) -> +5v
- C6 pad 2: Net-(C6-Pad2) -> A0
- C7 pad 1: GND -> A1
- C7 pad 2: Net-(C7-Pad2) -> GND
- C8 pad 1: GND -> A2
- C8 pad 2: Net-(C8-Pad2) -> GND
- C9 pad 1: Net-(C8-Pad2) -> GND
- C9 pad 2: Net-(U1-VBAT) -> Net-(C9-Pad2)
- I2C2_conn1 pad 1: +3v3 -> +5v
- I2C2_conn1 pad 2: Net-(I2C2_conn1-Pad2) -> UART8_TX
- I2C2_conn1 pad 3: Net-(I2C2_conn1-Pad3) -> UART8_RX
- I2C2_conn2 pad 2: I2C2_SLC -> Net-(JP3-B)
- I2C2_conn2 pad 3: I2C2_SDA -> Net-(U3-CANH)
- I2C2_conn3 pad 1: +5v -> +3v3
- I2C2_conn3 pad 2: UART8_TX -> Net-(I2C2_conn3-Pad2)
- I2C2_conn3 pad 3: UART8_RX -> Net-(I2C2_conn3-Pad3)
- I2C2_conn4 pad 2: Net-(U3-CANH) -> I2C2_SLC
- I2C2_conn4 pad 3: Net-(JP3-B) -> I2C2_SDA
- J10 pad 1: IN1_M1 -> A0
- J10 pad 2: IN2_M1 -> A1
- J10 pad 3: FS1 -> A2
- J10 pad 4: ENC_A_M1_mk -> A3
- J10 pad 5: ENC_B_M1_mk -> A4
- J11 pad 1: IN1_M2 -> +3v3
- J11 pad 2: IN2_M2 -> CLK
- J11 pad 3: FS2 -> SWDIO
- J11 pad 4: ENC_A_M2_mk -> NRST
- J11 pad 5: ENC_B_M2_mk -> GND
- J12 pad 1: IN1_M3 -> IN1_M4
- J12 pad 2: IN2_M3 -> IN2_M4
- J12 pad 3: FS3 -> FS4
- J12 pad 4: ENC_A_M3_mk -> ENC_A_M4_mk
- J12 pad 5: ENC_B_M3_mk -> ENC_B_M4_mk
- J13 pad 1: IN1_M5 -> IN1_M1
- J13 pad 2: IN2_M5 -> IN2_M1
- J13 pad 3: FS5 -> FS1
- J13 pad 4: ENC_A_M5_mk -> ENC_A_M1_mk
- J13 pad 5: ENC_B_M5_mk -> ENC_B_M1_mk
- J14 pad 1: IN1_M6 -> IN1_M2
- J14 pad 2: IN2_M6 -> IN2_M2
- J14 pad 3: FS6 -> FS2
- J14 pad 4: ENC_A_M6_mk -> ENC_A_M2_mk
- J14 pad 5: ENC_B_M6_mk -> ENC_B_M2_mk
- J2 pad 1: D33 -> +3v3
- J2 pad 2: D34 -> SDIO_D0
- J2 pad 3: D35 -> SDIO_CK
- J2 pad 4: D36 -> SDIO_CMD
- J2 pad 5: D37 -> GND
- J3 pad 1: A0 -> +3v3
- J3 pad 2: A1 -> SPI1_SCK
- J3 pad 3: A2 -> SPI1_MISO
- J3 pad 4: A3 -> SPI1_MOSI
- J3 pad 5: A4 -> GND
- J4 pad 1: D0 -> +3v3
- J4 pad 2: D1 -> SPI3_SCK
- J4 pad 3: D2 -> SPI3_MISO
- J4 pad 4: D3 -> SPI3_MOSI
- J4 pad 5: D4 -> GND
- J5 pad 1: D11 -> +3v3
- J5 pad 2: D12 -> SPI4_SCK
- J5 pad 3: D13 -> SPI4_MISO
- J5 pad 4: D14 -> SPI4_MOSI
- J5 pad 5: D15 -> GND
- J6 pad 1: D22 -> D0
- J6 pad 10: D31 -> D9
- J6 pad 11: D32 -> D10
- J6 pad 2: D23 -> D1
- J6 pad 3: D24 -> D2
- J6 pad 4: D25 -> D3
- J6 pad 5: D26 -> D4
- J6 pad 6: D27 -> D5
- J6 pad 7: D28 -> D6
- J6 pad 8: D29 -> D7
- J6 pad 9: D30 -> D8
- J9 pad 1: IN1_M4 -> D22
- J9 pad 2: IN2_M4 -> D23
- J9 pad 3: FS4 -> D24
- J9 pad 4: ENC_A_M4_mk -> D25
- J9 pad 5: ENC_B_M4_mk -> D26
- R1 pad 1: +3v3 -> BOOT0
- R1 pad 2: Data -> GND
- R10 pad 1: NRST -> PH0
- R10 pad 2: +3v3 -> PH1
- R13 pad 1: +3v3 -> A0
- R13 pad 2: ENC_B_M1_mk -> Net-(U1-PF3)
- R14 pad 1: ENC_A_M1_mk -> A1
- R14 pad 2: +3v3 -> Net-(U1-PF4)
- R15 pad 1: +3v3 -> A2
- R15 pad 2: ENC_A_M6_mk -> Net-(U1-PF5)
- R16 pad 1: ENC_B_M6_mk -> +3v3
- R16 pad 2: +3v3 -> ENC_A_M6_mk
- R17 pad 1: Net-(C6-Pad2) -> ENC_B_M6_mk
- R17 pad 2: Net-(U1-VCAP_1) -> +3v3
- R18 pad 1: Net-(C7-Pad2) -> Net-(C9-Pad2)
- R18 pad 2: Net-(U1-VCAP_2) -> Net-(U1-VCAP_1)
- R19 pad 1: +3v3 -> Net-(C10-Pad2)
- R19 pad 2: Net-(C8-Pad2) -> Net-(U1-VCAP_2)
- R2 pad 1: BOOT0 -> +3v3
- R2 pad 2: GND -> Data
- R20 pad 2: SDIO_CMD -> Net-(C11-Pad2)
- R21 pad 1: +3v3 -> ENC_A_M5_mk
- R21 pad 2: ENC_A_M2_mk -> +3v3
- R22 pad 1: +3v3 -> ENC_B_M5_mk
- R22 pad 2: ENC_B_M2_mk -> +3v3
- R23 pad 1: ENC_A_M4_mk -> +3v3
- R23 pad 2: +3v3 -> ENC_A_M2_mk
- R24 pad 1: ENC_B_M4_mk -> +3v3
- R24 pad 2: +3v3 -> ENC_B_M2_mk
- R25 pad 1: A0 -> ENC_A_M1_mk
- R25 pad 2: Net-(U1-PF3) -> +3v3
- R26 pad 1: A1 -> +3v3
- R26 pad 2: Net-(U1-PF4) -> ENC_B_M1_mk
- R27 pad 1: A2 -> A5
- R27 pad 2: Net-(U1-PF5) -> Net-(U1-PB0)
- R28 pad 1: +3v3 -> A6
- R28 pad 2: ENC_A_M3_mk -> Net-(U1-PB1)
- R29 pad 1: +3v3 -> A3
- R29 pad 2: ENC_B_M3_mk -> Net-(U1-PC4)
- R3 pad 1: TX_EN -> Net-(R3-Pad1)
- R3 pad 2: GND -> BOOT1
- R30 pad 1: ENC_A_M5_mk -> A4
- R30 pad 2: +3v3 -> Net-(U1-PC5)
- R31 pad 1: ENC_B_M5_mk -> DAC
- R31 pad 2: +3v3 -> GND
- R32 pad 1: A3 -> +3v3
- R32 pad 2: Net-(U1-PC4) -> ENC_A_M3_mk
- R33 pad 1: A6 -> +3v3
- R33 pad 2: Net-(U1-PB1) -> ENC_B_M3_mk
- R34 pad 1: +3v3 -> ENC_A_M4_mk
- R34 pad 2: SDIO_D0 -> +3v3
- R35 pad 1: A4 -> ENC_B_M4_mk
- R35 pad 2: Net-(U1-PC5) -> +3v3
- R36 pad 1: A5 -> Net-(J1-SHIELD)
- R36 pad 2: Net-(U1-PB0) -> GND
- R37 pad 1: DAC -> GND
- R37 pad 2: GND -> Net-(J1-CC1)
- R38 pad 1: Net-(U3-CANH) -> GND
- R38 pad 2: Net-(JP3-A) -> Net-(J1-CC2)
- R39 pad 1: Net-(J1-SHIELD) -> +3v3
- R39 pad 2: GND -> SDIO_CMD
- R4 pad 1: +3v3 -> TX_EN
- R4 pad 2: USART6_RX -> GND
- R40 pad 1: GND -> +3v3
- R40 pad 2: Net-(J1-CC1) -> SDIO_D0
- R41 pad 1: GND -> +3v3
- R41 pad 2: Net-(J1-CC2) -> I2C1_SCL
- R42 pad 2: I2C1_SCL -> I2C1_SDA
- R43 pad 1: +3v3 -> Net-(U3-CANH)
- R43 pad 2: I2C1_SDA -> Net-(JP3-A)
- R45 pad 1: Net-(I2C2_conn1-Pad2) -> Net-(I2C2_conn3-Pad2)
- R47 pad 1: Net-(I2C2_conn1-Pad3) -> Net-(I2C2_conn3-Pad3)
- R5 pad 1: Net-(R5-Pad1) -> +3v3
- R5 pad 2: BOOT1 -> Net-(R3-Pad1)
- R50 pad 1: +3v3 -> D37
- R50 pad 2: I2C2_SLC -> Net-(D4-A)
- R51 pad 1: +3v3 -> D38
- R51 pad 2: I2C2_SDA -> Net-(D5-A)
- R52 pad 1: D37 -> +3v3
- R52 pad 2: Net-(D5-A) -> Net-(D3-A)
- R53 pad 1: D38 -> +3v3
- R53 pad 2: Net-(D6-A) -> I2C3_SCL
- R54 pad 2: Net-(D7-A) -> I2C3_SDA
- R6 pad 1: PH0 -> GND
- R6 pad 2: PH1 -> Net-(R3-Pad1)
- R7 pad 1: PH1 -> +3v3
- R7 pad 2: Net-(C3-Pad2) -> USART6_RX
- R8 pad 1: +3v3 -> PH1
- R8 pad 2: Net-(R5-Pad1) -> Net-(C3-Pad2)
- R9 pad 1: GND -> NRST
- R9 pad 2: Net-(R5-Pad1) -> +3v3
- SW1 pad 1: NRST -> Net-(U1-PG12)
- SW2 pad 1: Net-(U1-PG12) -> NRST
Routing:
- net NRST: track 19.1 -> 0.00 mm
- net +3v3: track 14.8 -> 0.00 mm
- net GND: track 12.1 -> 0.00 mm
- net VDDA: track 8.72 -> 0.00 mm
- net VREF+: track 8.26 -> 0.00 mm
- net Net-(C4-Pad1): track 7.62 -> 0.00 mm
- net Net-(C5-Pad1): track 7.29 -> 0.00 mm
- net (no net): track 6.71 -> 0.00 mm
- net Net-(U1-PDR_ON): track 5.76 -> 0.00 mm
- net PC14: track 5.34 -> 0.00 mm
- net Net-(U1-PG12): track 5.25 -> 0.00 mm
- net PC15: track 5.13 -> 0.00 mm
- net Net-(C3-Pad2): track 4.51 -> 0.00 mm
- net Net-(C8-Pad2): track 4.08 -> 0.00 mm
- net Net-(U1-VBAT): track 3.53 -> 0.00 mm
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Other:
- board outline added: 100 x 100 mm

Commit message: c
Parts:
- moved J15 133.3 mm to (122.7, 87.7)
- moved J16 130.5 mm to (136.4, 130.0), turned to 90 degrees
- moved J12 122.3 mm to (121.9, 111.9)
- moved J17 107.8 mm to (165.2, 130.3), turned to 90 degrees
- moved J14 104.7 mm to (147.8, 74.4), turned to 90 degrees
- moved J13 75.2 mm to (173.1, 74.6), turned to 90 degrees
Routing:
- net IN1_M3: track 0.00 -> 27.0 mm
- net IN2_M3: track 0.00 -> 22.0 mm
- net FS3: track 0.00 -> 20.2 mm

Commit message: Дорожки
Parts:
- moved SW2 159.3 mm to (109.2, 112.1)
- moved CN1 157.0 mm to (108.8, 91.7), turned to -90 degrees
- moved SW1 155.4 mm to (109.3, 82.7), turned to 180 degrees
- moved J8 152.5 mm to (105.5, 56.0), turned to 90 degrees
- moved DynamixelCon1 152.2 mm to (110.2, 71.9), turned to 180 degrees
- moved J6 151.0 mm to (104.9, 118.8)
- moved D4 141.1 mm to (125.5, 55.3), turned to 180 degrees
- moved D5 140.7 mm to (125.5, 58.5), turned to 180 degrees
- moved J10 140.0 mm to (127.7, 149.1), turned to 90 degrees
- moved R50 138.4 mm to (122.2, 55.4)
- moved R51 138.4 mm to (122.2, 58.3)
- moved R46 135.3 mm to (113.8, 94.3)
- moved R44 134.6 mm to (113.8, 92.3)
- moved R42 134.1 mm to (112.8, 98.9)
- moved R41 134.0 mm to (112.9, 96.9)
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Connections:
- I2C2_conn1 pad 2: UART8_TX -> UART8_RX
- I2C2_conn1 pad 3: UART8_RX -> UART8_TX
- I2C2_conn4 pad 2: I2C2_SLC -> I2C2_SDA
- I2C2_conn4 pad 3: I2C2_SDA -> I2C2_SLC
- R48 pad 2: I2C2_SLC -> I2C2_SDA
- R49 pad 2: I2C2_SDA -> I2C2_SLC
Routing:
- net IN1_M3: track 27.0 -> 0.00 mm
- net IN2_M3: track 22.0 -> 0.00 mm
- net FS3: track 20.2 -> 0.00 mm
- net Net-(JP3-B): track 0.00 -> 3.13 mm
- net Net-(J1-SHIELD): track 0.00 -> 0.52 mm

Commit message: 2i
Parts:
- moved C22 91.6 mm to (132.6, 97.7), turned to 45 degrees
- moved C12 86.9 mm to (139.9, 111.7), turned to -135 degrees
- moved C21 84.1 mm to (139.8, 93.8), turned to -135 degrees
- moved C14 82.3 mm to (145.1, 116.5), turned to -45 degrees
- moved C20 80.1 mm to (143.8, 90.4), turned to -135 degrees
- moved C15 74.1 mm to (153.9, 117.8), turned to -135 degrees
- moved CN1 71.9 mm to (170.8, 55.2), turned to 180 degrees
- moved I2C2_conn3 69.6 mm to (159.8, 55.2), turned to 180 degrees
- moved C19 66.8 mm to (159.0, 91.1), turned to 135 degrees
- moved C16 65.6 mm to (159.1, 112.2), turned to 45 degrees
- moved R44 65.0 mm to (170.2, 60.1), turned to -90 degrees
- moved R41 64.8 mm to (165.6, 59.3), turned to -90 degrees
- moved R42 64.4 mm to (163.6, 59.2), turned to -90 degrees
- moved R46 64.3 mm to (168.2, 60.2), turned to -90 degrees
- moved R45 62.6 mm to (160.6, 60.3), turned to -90 degrees
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Routing:
- net DAC: track 0.00 -> 30.0 mm
- net Net-(U1-PF3): track 0.00 -> 16.6 mm
- net A5: track 0.00 -> 16.0 mm
- net A4: track 0.00 -> 15.9 mm
- net A3: track 0.00 -> 15.9 mm
- net A6: track 0.00 -> 15.9 mm
- net BOOT1: track 0.00 -> 14.6 mm
- net A2: track 0.00 -> 14.5 mm
- net Net-(U1-PF4): track 0.00 -> 14.5 mm
- net A1: track 0.00 -> 14.0 mm
- net Net-(U1-PF5): track 0.00 -> 12.2 mm
- net A0: track 0.00 -> 11.2 mm
- net Net-(U1-PB1): track 0.00 -> 8.74 mm
- net PH0: track 0.00 -> 8.32 mm
- net Net-(U1-PB0): track 0.00 -> 7.28 mm
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
Commit message: трассировка
Parts:
- moved C38 17.2 mm to (182.1, 96.9), turned to -90 degrees
- moved J13 10.8 mm to (177.4, 77.2), turned to -90 degrees
- moved C39 5.57 mm to (196.7, 112.3)
- moved R25 5.15 mm to (170.1, 79.8), turned to 0 degrees
- moved C12 5.00 mm to (137.1, 115.7)
- moved L1 4.59 mm to (145.0, 120.9)
- moved R23 3.79 mm to (130.8, 80.4)
- moved R24 3.79 mm to (127.7, 80.4)
- moved J14 3.79 mm to (138.1, 77.8)
- moved R26 2.81 mm to (167.0, 79.8), turned to 0 degrees
- moved C32 2.59 mm to (146.1, 118.6)
- moved C33 2.59 mm to (147.2, 117.4)
- moved L2 2.57 mm to (143.9, 119.8)
- moved C24 1.95 mm to (163.3, 118.8)
- moved C27 1.95 mm to (160.4, 121.7)
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Routing:
- net DAC: track 30.0 -> 0.00 mm
- net GND: track 0.00 -> 28.0 mm
- net Net-(U1-PF3): track 16.6 -> 0.00 mm
- net A5: track 16.0 -> 0.00 mm
- net A4: track 15.9 -> 0.00 mm
- net A3: track 15.9 -> 0.00 mm
- net A6: track 15.9 -> 0.00 mm
- net BOOT1: track 14.6 -> 0.00 mm
- net A2: track 14.5 -> 0.00 mm
- net Net-(U1-PF4): track 14.5 -> 0.00 mm
- net A1: track 14.0 -> 0.00 mm
- net Net-(U1-PF5): track 12.2 -> 0.00 mm
- net A0: track 11.2 -> 0.00 mm
- net Net-(U1-PG12): track 0.00 -> 10.8 mm
- net NRST: track 0.00 -> 10.5 mm
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Other:
- board text added: "1) Кварц 2) Питание 3) АЦП 4) Интерфейсы и обвязка"

Commit message: tras
Parts:
- moved J9 57.5 mm to (183.9, 109.3)
- moved C39 27.0 mm to (172.0, 101.4), turned to 90 degrees
- moved J10 26.1 mm to (130.8, 148.9)
- moved C34 24.4 mm to (193.2, 63.3)
- moved J1 24.4 mm to (197.0, 69.4)
- moved R36 24.4 mm to (193.4, 75.8)
- moved R37 24.4 mm to (190.7, 73.0)
- moved R38 24.4 mm to (190.7, 65.8)
- moved U2 24.4 mm to (187.3, 69.3)
- moved R52 22.2 mm to (174.8, 96.3), turned to 0 degrees
- moved D3 21.5 mm to (174.9, 94.5), turned to 180 degrees
- moved con1 20.1 mm to (174.7, 104.2), turned to 180 degrees
- moved C8 17.6 mm to (125.4, 133.1), turned to -135 degrees
- moved C7 15.8 mm to (123.7, 131.6), turned to 45 degrees
- moved R15 14.8 mm to (127.3, 130.5), turned to 45 degrees
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Routing:
- net +3v3: track 9.38 -> 324.9 mm
- net GND: track 28.0 -> 69.2 mm
- net Net-(U1-PG12): track 10.8 -> 0.00 mm
- net IN2_M5: track 0.00 -> 10.1 mm, vias 0 -> 1
- net FS5: track 0.00 -> 9.64 mm, vias 0 -> 1
- net VREF+: track 0.00 -> 9.19 mm
- net NRST: track 10.5 -> 1.54 mm, vias 0 -> 1
- net Net-(C5-Pad1): track 8.51 -> 0.00 mm
- net D10: track 0.00 -> 8.40 mm, vias 0 -> 1
- net VDDA: track 0.00 -> 7.87 mm
- net Net-(C4-Pad1): track 7.72 -> 0.00 mm
- net PH0: track 0.00 -> 7.39 mm
- net ENC_A_M5_mk: track 0.00 -> 6.91 mm, vias 0 -> 1
- net PH1: track 0.00 -> 6.35 mm
- net PC15: track 0.00 -> 6.27 mm
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